File: hadbadge2019.kicad_pcb (KiCad board)
At the start: 4 copper layers, 80 x 100 mm, 137 parts, among them J1 Conn_02x04_Odd_Even, J2 USB_B_Micro, J3 HDMI_A_1.4, J4 FH26W-45S-0.3SHW(60), J5 Conn_02x16_Odd_Even, J6 Conn_01x02, Q1 AO3400, SW1 Up, SW2 Down, SW3 Left, SW4 Right, SW5 A, SW6 B, SW7 Select, SW8 Start, U1 LFE5UM-45F, U10 NS8002, U2 25LCxxx, U3 M3406, U4 XC6206P25, U5 XC6206P12, U6 ME2108A33M3, U7 ME2108A50M3, U8 LY68L6400SLIT, U9 LY68L6400SLIT, X1 X1G004481001400

Commit message: Proto 1
Parts:
- removed the C4 at (126.6, 82.8)
- removed C48, C49, C50: 10u, Capacitor_SMD:C_0805_2012Metric
- removed the D4 at (88.7, 56.7)
- removed the R32 at (91.8, 49.4)
- removed the R37 at (125.8, 64.6)
- removed the TP12 at (111.8, 86.6)
- added C26: 10u, Capacitor_SMD:C_0805_2012Metric, B.Cu at (90.8, 37.6)
- added C27: 10u, Capacitor_SMD:C_0805_2012Metric, B.Cu at (96.1, 41.9)
- added C28: 10u, Capacitor_SMD:C_0805_2012Metric, B.Cu at (93.9, 38.6)
- added C7: 100n, Capacitor_SMD:C_0603_1608Metric, B.Cu at (126.6, 82.8)
- added D1: SS12, Diode_SMD:D_SMA, B.Cu at (93.8, 45.8)
- added D10: LED, LED_SMD:LED_0603_1608Metric, F.Cu at (139.6, 79.7)
- added D5: LED, LED_SMD:LED_0603_1608Metric, F.Cu at (139.6, 70.8)
- added D6: LED, LED_SMD:LED_0603_1608Metric, F.Cu at (139.6, 72.6)
- added D7: LED, LED_SMD:LED_0603_1608Metric, F.Cu at (139.6, 74.4)
- added D8: LED, LED_SMD:LED_0603_1608Metric, F.Cu at (139.6, 76.2)
- added D9: LED, LED_SMD:LED_0603_1608Metric, F.Cu at (139.6, 78.0)
- added R1: 4K7, Resistor_SMD:R_0603_1608Metric, B.Cu at (125.8, 64.6)
- added R21: 0, Resistor_SMD:R_0603_1608Metric, B.Cu at (96.9, 38.5)
- added R41: 470, Resistor_SMD:R_0603_1608Metric, B.Cu at (135.9, 71.2)
- added R42: 470, Resistor_SMD:R_0603_1608Metric, B.Cu at (135.9, 72.7)
- added R43: 470, Resistor_SMD:R_0603_1608Metric, B.Cu at (135.9, 74.2)
- added R44: 470, Resistor_SMD:R_0603_1608Metric, B.Cu at (135.9, 75.7)
- added R45: 470, Resistor_SMD:R_0603_1608Metric, B.Cu at (135.9, 77.2)
- added R46: 470, Resistor_SMD:R_0603_1608Metric, B.Cu at (135.9, 78.7)
- added SW9: SW_SPDT_shielded, lib:Korean_Hroparts_K3_1296S, B.Cu at (85.3, 17.8)
- added TP7: TestPoint, TestPoint:TestPoint_Pad_D1.0mm, F.Cu at (111.8, 86.6)
- L1: value 2u2 -> SWPA252010S4R7MT; footprint Inductor_SMD:L_1206_3216Metric_Pad1.42x1.75mm_HandSolder -> lib:SWPA25xx
- L2, L3: value 47u -> SWPA6045S470MT; footprint Inductor_SMD:L_1206_3216Metric_Pad1.42x1.75mm_HandSolder -> lib:SWPA60xx
- moved L2 18.5 mm to (86.2, 42.0), turned to 90 degrees
- moved L3 12.8 mm to (96.4, 56.9), turned to 270 degrees
- moved U7 12.0 mm to (92.7, 42.2)
- moved L1 0.42 mm to (121.5, 51.5)
- renumbered C52 to C1, C46 to C10, C47 to C11, C8 to C12, C10 to C13, C12 to C14, C14 to C15, C22 to C18, C23 to C19, C51 to C2, C26 to C20, C27 to C21, C1 to C22, C28 to C23, C29 to C24, C30 to C25, C31 to C29, C57 to C3, C32 to C30, C33 to C31, C34 to C32, C35 to C33, C54 to C34, C36 to C35, C37 to C36, C38 to C37, C39 to C38, C40 to C39, C53 to C4, C55 to C40, C56 to C44, C44 to C45, C45 to C46, C2 to C47, C3 to C6, C6 to C8, C7 to C9, D1 to D2, D2 to D3, D3 to D4, J6 to J3, J3 to J4, J4 to J5, J5 to J6, R4 to R10, R5 to R11, R6 to R12, R7 to R13, R8 to R14, R9 to R15, R10 to R16, R28 to R17, R11 to R18, R12 to R19, R38 to R2, R29 to R20, R13 to R22, R30 to R23, R31 to R24, R14 to R25, R15 to R26, R16 to R27, R34 to R28, R17 to R29, R39 to R3, R18 to R30, R35 to R31, R19 to R32, R20 to R33, R21 to R34, R22 to R35, R23 to R36, R24 to R37, R25 to R38, R26 to R39, R40 to R4, R27 to R40, R36 to R5, R33 to R6, R1 to R7, R2 to R8, R3 to R9, TP6 to TP1, TP15 to TP10, TP1 to TP11, TP2 to TP12, TP3 to TP13, TP4 to TP14, TP5 to TP15, TP7 to TP2, TP8 to TP3, TP9 to TP4, TP10 to TP5, TP11 to TP6, TP13 to TP8, TP14 to TP9, U8 to U2, U9 to U3, U2 to U4, U3 to U5, U4 to U6, U5 to U8, U6 to U9
Connections:
- BT1 pad 1: VBAT -> VBAT_ALWON
- D2 pad 2: Net-(D1-Pad2) -> Net-(D2-Pad2)
- J1 pad 2: VBAT -> VBAT_ALWON
- L3 pad 1: Net-(D4-Pad2) -> Net-(D2-Pad2)
- U1 pad C4: Net-(U1-PadC4) -> LED4
- U1 pad C5: Net-(U1-PadC5) -> LED5
- U1 pad C6: Net-(U1-PadC6) -> LED6
- U1 pad D20: Net-(U1-PadD20) -> PWMOUT
- U1 pad D3: Net-(U1-PadD3) -> LED3
- U1 pad E3: Net-(U1-PadE3) -> LED2
- U1 pad F3: Net-(U1-PadF3) -> LED1
- U1 pad H3: Net-(U1-PadH3) -> LCD_BLEN
- U7 pad 2: Net-(D4-Pad2) -> Net-(D1-Pad2)
- U9 pad 2: Net-(D1-Pad2) -> Net-(D2-Pad2)
Routing:
- net VBAT_ALWON: track 0.00 -> 77.0 mm
- net LCD_BLEN: track 2.19 -> 61.5 mm, vias 0 -> 2
- net PWMOUT: track 0.00 -> 16.7 mm, vias 0 -> 1
- net 5V: track 96.6 -> 112.3 mm
- net GND: track 203.1 -> 217.9 mm, vias 54 -> 57
- net LED1: track 0.00 -> 8.55 mm, vias 0 -> 1
- net VBAT: track 208.2 -> 216.1 mm
- net LED2: track 0.00 -> 7.13 mm, vias 0 -> 1
- net LED3: track 0.00 -> 5.70 mm, vias 0 -> 1
- net LED6: track 0.00 -> 5.46 mm, vias 0 -> 1
- net Net-(D2-Pad2): track 0.00 -> 5.46 mm
- net LED5: track 0.00 -> 4.97 mm, vias 0 -> 1
- net Net-(D4-Pad2): track 4.86 -> 0.00 mm
- net LED4: track 0.00 -> 4.67 mm, vias 0 -> 1
- net Net-(D1-Pad2): track 5.46 -> 8.55 mm
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Other:
- board text added: "1V1"
- board text added: "1V1 serdes"
- board text added: "2V5"
- board text added: "3V3 boost"
- board text added: "5V boost"
- board text added: "8/16MB RAM"
- board text added: "<- ON"
- board text added: "DOT MATRIX MONO SOUND"
- board text added: "GND VIO IO2 IO1 IO4 IO3 ETC"
- board text added: "Hackaday Supercon 2019 Badge Proto v2 Spritesmods.com"
- board text added: "JTAG: GND VBAT NC VIO TDO TMS TCK TDI"
- board text added: "Relaxen und watchen das blinkenlichten."
- board text added: "ToDo: replace USB footprint for something sane"
- board text removed: "HDMI-ish"

Commit message: New design
Parts:
- added J10: Conn_01x02_Male, Connector_PinHeader_2.54mm:PinHeader_1x02_P2.54mm_Vertical, F.Cu at (146.7, 22.0)
- added J7: Conn_02x03_Odd_Even, Connector_PinSocket_2.54mm:PinSocket_2x03_P2.54mm_Vertical, F.Cu at (121.1, 27.0)
- added J8: Conn_02x03_Odd_Even, Connector_PinSocket_2.54mm:PinSocket_2x03_P2.54mm_Vertical, F.Cu at (148.0, 27.0)
- added J9: Conn_01x02_Male, Connector_PinHeader_2.54mm:PinHeader_1x02_P2.54mm_Vertical, F.Cu at (119.8, 22.0)
- C1: value C -> 100n
- C2: value C -> 100n; moved to B.Cu
- C39, C4, C41, R33, R34, R35, R36, R37, R38, TP13, TP14, TP15: moved to B.Cu
- R10: value NS -> 4K7
- R15: value NS -> 0
- R16: value 0 -> NS
- R6: value R -> 0
- R9: value 4K7 -> NS
- SW1, SW2, SW3, SW4, SW5, SW6, SW7, SW8: footprint Button_Switch_THT:SW_PUSH_6mm -> Button_Switch_SMD:SW_Push_1P1T_NO_6x6mm_H9.5mm
- U10, U4: moved to F.Cu
- U2, U3: footprint Package_SO:SO-8_5.3x6.2mm_P1.27mm -> Package_SO:SSOP-8_3.9x5.05mm_P1.27mm
- moved C12 206.4 mm to (307.6, 142.7)
- moved C20 206.4 mm to (322.6, 148.6)
- moved R11 206.4 mm to (307.2, 147.6)
- moved R12 206.4 mm to (299.8, 144.9)
- moved TP11 206.4 mm to (307.7, 145.5)
- moved R2 201.5 mm to (317.5, 128.0)
- moved C21 175.4 mm to (258.3, 165.6)
- moved C22 175.4 mm to (262.3, 159.4)
- moved C23 175.4 mm to (256.0, 160.8)
- moved C24 175.4 mm to (251.0, 167.8)
- moved C25 175.4 mm to (256.4, 168.2)
- moved C26 175.4 mm to (227.8, 147.1)
- moved C27 175.4 mm to (233.1, 151.4)
- moved C28 175.4 mm to (230.9, 148.1)
- moved C29 175.4 mm to (249.9, 161.8)
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Connections:
- J1 pad 3: Net-(J1-Pad3) -> (no net)
- J6 pad 3: GENIO_1 -> (no net)
- J6 pad 4: GENIO_2 -> (no net)
- J6 pad 5: GENIO_3 -> (no net)
- J6 pad 6: GENIO_4 -> (no net)
- J6 pad 7: GENIO_5 -> (no net)
- J6 pad 8: GENIO_6 -> (no net)
- J6 pad 9: GENIO_7 -> (no net)
- R25 pad 1: USB_PU -> (no net)
- R5 pad 2: PWMOUT -> (no net)
- SW9 pad 3: Net-(SW9-Pad3) -> (no net)
- U1 pad A12: Net-(U1-PadA12) -> (no net)
- U1 pad A13: Net-(U1-PadA13) -> (no net)
- U1 pad A14: RAM1_SIO3 -> (no net)
- U1 pad A15: RAM1_SCLK -> (no net)
- U1 pad A16: RAM1_CE -> (no net)
- U1 pad A17: RAM1_SIO2 -> (no net)
- U1 pad A18: RAM2_SCLK -> (no net)
- U1 pad A19: RAM2_CE -> (no net)
- U1 pad B12: Net-(U1-PadB12) -> (no net)
- U1 pad B13: Net-(U1-PadB13) -> (no net)
- U1 pad B15: RAM1_SIO0 -> (no net)
- U1 pad B16: RAM1_SIO1 -> (no net)
- U1 pad B17: RAM2_SIO3 -> (no net)
- U1 pad B18: RAM2_SIO0 -> (no net)
- U1 pad B19: RAM2_SIO1 -> (no net)
- U1 pad B20: RAM2_SIO2 -> (no net)
- U1 pad C1: GENIO_7 -> BTN_DOWN
- U1 pad C10: Net-(U1-PadC10) -> (no net)
- U1 pad C11: BTN_B -> (no net)
- U1 pad C12: Net-(U1-PadC12) -> (no net)
- U1 pad C13: Net-(U1-PadC13) -> (no net)
- U1 pad C14: Net-(U1-PadC14) -> (no net)
- U1 pad C15: Net-(U1-PadC15) -> (no net)
- U1 pad C16: Net-(U1-PadC16) -> (no net)
- U1 pad C17: Net-(U1-PadC17) -> (no net)
- U1 pad C18: Net-(U1-PadC18) -> (no net)
- U1 pad C20: BTN_START -> RAM1_SIO2
- U1 pad C8: Net-(U1-PadC8) -> (no net)
- U1 pad C9: BTN_A -> (no net)
- U1 pad D1: GENIO_5 -> BTN_A
- U1 pad D10: Net-(U1-PadD10) -> (no net)
- U1 pad D11: Net-(U1-PadD11) -> (no net)
- U1 pad D12: Net-(U1-PadD12) -> (no net)
- U1 pad D13: Net-(U1-PadD13) -> (no net)
- U1 pad D14: Net-(U1-PadD14) -> (no net)
- U1 pad D15: Net-(U1-PadD15) -> (no net)
- U1 pad D16: Net-(U1-PadD16) -> (no net)
- U1 pad D17: Net-(U1-PadD17) -> (no net)
- U1 pad D18: Net-(U1-PadD18) -> (no net)
- U1 pad D19: Net-(U1-PadD19) -> RAM1_SIO1
- U1 pad D2: GENIO_6 -> BTN_SELECT
- U1 pad D20: PWMOUT -> RAM1_CE
- U1 pad D5: Net-(U1-PadD5) -> (no net)
- U1 pad D6: Net-(U1-PadD6) -> (no net)
- U1 pad D7: Net-(U1-PadD7) -> (no net)
- U1 pad D8: Net-(U1-PadD8) -> (no net)
- U1 pad D9: Net-(U1-PadD9) -> (no net)
- U1 pad E1: GENIO_3 -> BTN_START
- U1 pad E10: Net-(U1-PadE10) -> (no net)
- U1 pad E11: Net-(U1-PadE11) -> (no net)
- U1 pad E12: Net-(U1-PadE12) -> (no net)
- U1 pad E13: Net-(U1-PadE13) -> (no net)
- U1 pad E14: Net-(U1-PadE14) -> (no net)
- U1 pad E15: Net-(U1-PadE15) -> (no net)
- U1 pad E16: Net-(U1-PadE16) -> (no net)
- U1 pad E17: Net-(U1-PadE17) -> (no net)
- U1 pad E18: Net-(U1-PadE18) -> (no net)
- U1 pad E19: Net-(U1-PadE19) -> RAM1_SIO0
- U1 pad E2: GENIO_4 -> BTN_B
- U1 pad E20: Net-(U1-PadE20) -> RAM1_SCLK
- U1 pad E4: Net-(U1-PadE4) -> (no net)
- U1 pad E5: Net-(U1-PadE5) -> (no net)
- U1 pad E6: Net-(U1-PadE6) -> (no net)
- U1 pad E7: Net-(U1-PadE7) -> (no net)
- U1 pad E8: Net-(U1-PadE8) -> (no net)
- U1 pad E9: Net-(U1-PadE9) -> (no net)
- U1 pad F1: GENIO_1 -> BTN_UP
- U1 pad F11: VIO_PSRAM -> VIO
- U1 pad F12: VIO_PSRAM -> VIO
- U1 pad F16: Net-(U1-PadF16) -> (no net)
- U1 pad F17: Net-(U1-PadF17) -> (no net)
- U1 pad F18: Net-(U1-PadF18) -> (no net)
- U1 pad F19: Net-(U1-PadF19) -> RAM1_SIO3
- U1 pad F2: GENIO_2 -> BTN_RIGHT
- U1 pad F20: Net-(U1-PadF20) -> RAM2_CE
- U1 pad F4: Net-(U1-PadF4) -> (no net)
- U1 pad F5: Net-(U1-PadF5) -> (no net)
- U1 pad G1: LCD_RS -> LCD_FMARK
- U1 pad G16: Net-(U1-PadG16) -> (no net)
- U1 pad G18: Net-(U1-PadG18) -> (no net)
- U1 pad G19: Net-(U1-PadG19) -> RAM2_SIO1
- U1 pad G2: LCD_DB17 -> (no net)
- U1 pad G20: USB_VBUSDET -> RAM2_SIO2
- U1 pad G3: Net-(U1-PadG3) -> BTN_LEFT
- U1 pad G5: Net-(U1-PadG5) -> (no net)
- U1 pad H1: LCD_DB15 -> LCD_DB1
- U1 pad H14: VIO -> VIO_PSRAM
- U1 pad H15: VIO -> VIO_PSRAM
- U1 pad H16: Net-(U1-PadH16) -> (no net)
- U1 pad H17: Net-(U1-PadH17) -> (no net)
- U1 pad H18: Net-(U1-PadH18) -> (no net)
- U1 pad H2: LCD_RD -> LCD_RST
- U1 pad H20: USB_PU -> RAM2_SIO3
- U1 pad H4: Net-(U1-PadH4) -> (no net)
- U1 pad H5: Net-(U1-PadH5) -> (no net)
- U1 pad J1: LCD_CS -> LCD_DB3
- U1 pad J15: VIO -> VIO_PSRAM
- U1 pad J16: Net-(U1-PadJ16) -> (no net)
- U1 pad J17: Net-(U1-PadJ17) -> (no net)
- U1 pad J18: Net-(U1-PadJ18) -> (no net)
- U1 pad J19: USB_D+ -> RAM2_SCLK
- U1 pad J20: CLK -> RAM2_SIO0
- U1 pad J3: LCD_DB13 -> LCD_DB0
- U1 pad J4: Net-(U1-PadJ4) -> LCD_ID
- U1 pad J5: Net-(U1-PadJ5) -> (no net)
- U1 pad K1: LCD_DB16 -> LCD_DB7
- U1 pad K16: Net-(U1-PadK16) -> (no net)
- U1 pad K17: Net-(U1-PadK17) -> (no net)
- U1 pad K18: Net-(U1-PadK18) -> (no net)
- U1 pad K19: USB_D- -> (no net)
- U1 pad K2: LCD_WR -> LCD_DB5
- U1 pad K20: Net-(U1-PadK20) -> (no net)
- U1 pad K3: LCD_DB11 -> LCD_DB4
- U1 pad K4: LCD_DB9 -> LCD_DB2
- U1 pad K5: Net-(U1-PadK5) -> (no net)
- U1 pad L1: LCD_DB12 -> LCD_DB11
- U1 pad L16: Net-(U1-PadL16) -> HDMI_D2+
- U1 pad L17: Net-(U1-PadL17) -> HDMI_D2-
- U1 pad L18: Net-(U1-PadL18) -> (no net)
- U1 pad L19: BTN_SELECT -> (no net)
- U1 pad L2: LCD_DB14 -> LCD_DB9
- U1 pad L20: HDMI_HEAC+ -> HDMI_D1+
- U1 pad L3: Net-(U1-PadL3) -> LCD_DB8
- U1 pad L4: Net-(U1-PadL4) -> LCD_DB6
- U1 pad L5: Net-(U1-PadL5) -> (no net)
- U1 pad M1: LCD_DB8 -> LCD_DB13
- U1 pad M17: HDMI_CK- -> (no net)
- U1 pad M18: Net-(U1-PadM18) -> (no net)
- U1 pad M19: Net-(U1-PadM19) -> (no net)
- U1 pad M20: HDMI_HEAC- -> HDMI_D1-
- U1 pad M3: LCD_DB10 -> LCD_DB12
- U1 pad M4: LCD_DB5 -> LCD_DB10
- U1 pad M5: LCD_DB7 -> (no net)
- U1 pad N1: LCD_DB4 -> LCD_DB17
- U1 pad N16: HDMI_CK+ -> (no net)
- U1 pad N17: HDMI_D1+ -> (no net)
- U1 pad N18: Net-(U1-PadN18) -> (no net)
- U1 pad N2: LCD_DB6 -> LCD_DB15
- U1 pad N3: LCD_DB1 -> LCD_DB16
- U1 pad N4: LCD_DB3 -> LCD_DB14
- U1 pad N5: Net-(U1-PadN5) -> (no net)
- U1 pad P1: LCD_DB0 -> LCD_RS
- U1 pad P16: HDMI_D1- -> (no net)
- U1 pad P17: Net-(U1-PadP17) -> (no net)
- U1 pad P18: Net-(U1-PadP18) -> (no net)
- U1 pad P19: Net-(U1-PadP19) -> (no net)
- U1 pad P2: LCD_DB2 -> LCD_RD
- U1 pad P20: HDMI_D2+ -> HDMI_CK+
- U1 pad P3: LCD_ID -> LCD_CS
- U1 pad P4: LCD_FMARK -> LCD_WR
- U1 pad P5: LCD_RST -> (no net)
- U1 pad R1: Net-(U1-PadR1) -> (no net)
- U1 pad R16: Net-(U1-PadR16) -> (no net)
- U1 pad R17: Net-(U1-PadR17) -> (no net)
- U1 pad R18: Net-(U1-PadR18) -> HDMI_HEAC-
- U1 pad R20: HDMI_D2- -> HDMI_CK-
- U1 pad R3: Net-(U1-PadR3) -> (no net)
- U1 pad T1: Net-(U1-PadT1) -> (no net)
- U1 pad T16: Net-(U1-PadT16) -> (no net)
- U1 pad T17: Net-(U1-PadT17) -> (no net)
- U1 pad T18: Net-(U1-PadT18) -> (no net)
- U1 pad T19: Net-(U1-PadT19) -> HDMI_HEAC+
- U1 pad T2: Net-(U1-PadT2) -> (no net)
- U1 pad T20: BTN_DOWN -> (no net)
- U1 pad T3: Net-(U1-PadT3) -> (no net)
- U1 pad U1: Net-(U1-PadU1) -> (no net)
- U1 pad U16: Net-(U1-PadU16) -> (no net)
- U1 pad U17: Net-(U1-PadU17) -> (no net)
- U1 pad U18: BTN_UP -> (no net)
- U1 pad U19: BTN_LEFT -> (no net)
- U1 pad U2: Net-(U1-PadU2) -> (no net)
- U1 pad U20: BTN_RIGHT -> (no net)
- U1 pad V1: Net-(U1-PadV1) -> (no net)
- U1 pad W10: Net-(U1-PadW10) -> (no net)
- U1 pad W11: Net-(U1-PadW11) -> (no net)
- U1 pad W13: Net-(U1-PadW13) -> (no net)
- U1 pad W14: Net-(U1-PadW14) -> (no net)
- U1 pad W17: Net-(U1-PadW17) -> (no net)
- U1 pad W18: Net-(U1-PadW18) -> (no net)
- U1 pad W20: Net-(U1-PadW20) -> (no net)
- U1 pad Y14: Net-(U1-PadY14) -> (no net)
- U1 pad Y15: Net-(U1-PadY15) -> (no net)
- U1 pad Y16: Net-(U1-PadY16) -> (no net)
- U1 pad Y17: Net-(U1-PadY17) -> (no net)
- U1 pad Y19: Net-(U1-PadY19) -> (no net)
- X1 pad 3: CLK -> (no net)
Routing:
- net VBAT: track 216.1 -> 0.00 mm, vias 2 -> 0
- net GND: track 217.9 -> 65.3 mm, vias 57 -> 33
- net 5V: track 112.3 -> 0.00 mm, vias 3 -> 0
- net VBAT_ALWON: track 77.0 -> 0.00 mm
- net Net-(BT1-Pad2): track 68.0 -> 0.00 mm
- net GENIO_2: track 67.5 -> 0.00 mm
- net GENIO_4: track 64.7 -> 0.00 mm
- net GENIO_1: track 64.5 -> 0.00 mm
- net GENIO_6: track 61.8 -> 0.00 mm
- net GENIO_3: track 61.7 -> 0.00 mm
- net LCD_BLEN: track 61.5 -> 0.00 mm, vias 2 -> 0
- net VIO: track 65.8 -> 5.26 mm, vias 17 -> 3
- net 2V5: track 59.4 -> 0.00 mm, vias 7 -> 0
- net GENIO_8: track 58.9 -> 0.00 mm
- net GENIO_5: track 58.8 -> 0.00 mm
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- removed copper zone on Pwr.Cu, net 1V1
Other:
- board size 80 x 100 mm -> 96 x 145.5 mm
- board text added: "DOT MATRIX WITH MONO SOUND"
- board text removed: "DOT MATRIX MONO SOUND"

Commit message: WiP for proto 2
Parts:
- removed C27, C28: 10u, Capacitor_SMD:C_0805_2012Metric
- removed C29, C30: 1u, Capacitor_SMD:C_0603_1608Metric
- removed TP1, TP10, TP2, TP3, TP4, TP5, TP6, TP7, TP8, TP9: TestPoint, TestPoint:TestPoint_Pad_D1.0mm
- added R47: R, Resistor_SMD:R_0603_1608Metric, B.Cu at (138.8, 184.1)
- C10, C11: value 100n -> 10u; footprint Capacitor_SMD:C_0603_1608Metric -> Capacitor_SMD:C_0805_2012Metric
- C4: value 100n -> 22p; footprint Capacitor_SMD:C_0603_1608Metric -> Capacitor_SMD:C_0805_2012Metric
- C47, Q1, R39, R40, TP11: moved to B.Cu
- D1, D2: value SS12 -> MBRA210LT3
- J3: moved to F.Cu
- J6: footprint Connector_PinSocket_2.54mm:PinSocket_2x16_P2.54mm_Vertical -> Connector_PinSocket_2.54mm:PinSocket_2x16_P2.54mm_Horizontal
- L2, L3: value SWPA6045S470MT -> LQH3NPN2R2MJRL; footprint lib:SWPA60xx -> Inductor_SMD:L_Murata_DEM35xxC
- R21: value 0 -> 100K
- R22: value NS -> 0
- R23, R6: value 0 -> R
- U7: value ME2108A50M3 -> XR1151; footprint Package_TO_SOT_SMD:SOT-23 -> Package_TO_SOT_SMD:SOT-23-6
- U8: value XC6206P12 -> ESP-WROVER32; footprint Package_TO_SOT_SMD:SOT-23 -> RF_Module:ESP32-WROOM-32
- U9: value ME2108A33M3 -> XR1151; footprint Package_TO_SOT_SMD:SOT-23 -> Package_TO_SOT_SMD:SOT-23-6
- moved TP12 229.0 mm to (75.1, 75.8), turned to 90 degrees
- moved J2 228.0 mm to (75.9, 76.3), turned to 90 degrees
- moved R2 223.1 mm to (95.4, 149.0), turned to 0 degrees
- moved R32 220.0 mm to (82.1, 80.8), turned to 180 degrees
- moved D3 219.7 mm to (81.4, 73.1), turned to 90 degrees
- moved R27 219.7 mm to (82.1, 79.1), turned to 180 degrees
- moved R29 219.4 mm to (82.1, 77.4), turned to 180 degrees
- moved R30 219.2 mm to (82.1, 75.9), turned to 180 degrees
- moved D4 217.6 mm to (82.9, 73.1), turned to 90 degrees
- moved C20 215.6 mm to (108.0, 128.8), turned to 90 degrees
- moved C44 214.9 mm to (74.8, 125.7), turned to 90 degrees
- moved C12 212.1 mm to (96.2, 125.5)
- moved R11 211.4 mm to (96.0, 137.7)
- moved R28 210.2 mm to (74.8, 141.9), turned to 90 degrees
- moved TP11 209.6 mm to (98.2, 137.6)
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Connections:
- C1 pad 1: VIO_PSRAM -> VIO
- C10 pad 1: 1V1_SERDES -> Net-(C10-Pad1)
- C11 pad 1: 1V1_SERDES -> Net-(C10-Pad1)
- C2 pad 1: VIO_PSRAM -> VIO
- C4 pad 1: VIO_PSRAM -> Net-(C32-Pad1)
- C4 pad 2: GND -> Net-(C4-Pad2)
- D1 pad 1: Net-(C27-Pad1) -> Net-(C10-Pad1)
- R21 pad 1: 5V -> Net-(C4-Pad2)
- R21 pad 2: Net-(C27-Pad1) -> GND
- R22 pad 1: 1V1 -> 5V
- R22 pad 2: Net-(C30-Pad1) -> Net-(C10-Pad1)
- R23 pad 1: 1V1_SERDES -> Net-(C10-Pad1)
- R23 pad 2: Net-(C30-Pad1) -> Net-(R23-Pad2)
- R6 pad 1: VIO_PSRAM -> Net-(C32-Pad1)
- R6 pad 2: VIO -> Net-(C4-Pad2)
- SW9 pad 1: VBAT -> VBAT_ALWON
- SW9 pad 2: VBAT_ALWON -> VBAT
- U1 pad H14: VIO_PSRAM -> VIO
- U1 pad H15: VIO_PSRAM -> VIO
- U1 pad H3: LCD_BLEN -> (no net)
- U1 pad J15: VIO_PSRAM -> VIO
- U1 pad P5: (no net) -> LCD_BLEN
- U1 pad T15: 1V1_SERDES -> 1V1
- U1 pad T6: 1V1_SERDES -> 1V1
- U1 pad U15: 1V1_SERDES -> 1V1
- U1 pad U6: 1V1_SERDES -> 1V1
- U1 pad W4: Net-(TP1-Pad1) -> (no net)
- U1 pad W5: Net-(TP2-Pad1) -> (no net)
- U1 pad W8: Net-(TP7-Pad1) -> (no net)
- U1 pad W9: Net-(TP8-Pad1) -> (no net)
- U1 pad Y11: Net-(TP9-Pad1) -> (no net)
- U1 pad Y12: Net-(TP10-Pad1) -> (no net)
- U1 pad Y5: Net-(TP3-Pad1) -> (no net)
- U1 pad Y6: Net-(TP4-Pad1) -> (no net)
- U1 pad Y7: Net-(TP5-Pad1) -> (no net)
- U1 pad Y8: Net-(TP6-Pad1) -> (no net)
- U2 pad 8: VIO_PSRAM -> VIO
- U3 pad 8: VIO_PSRAM -> VIO
- U7 pad 1: GND -> Net-(D2-Pad2)
- U7 pad 2: Net-(D1-Pad2) -> GND
- U7 pad 3: Net-(C27-Pad1) -> Net-(C4-Pad2)
- U8 pad 1: GND -> (no net)
- U8 pad 2: Net-(C30-Pad1) -> (no net)
- U8 pad 3: VBAT -> (no net)
- U9 pad 1: GND -> Net-(D1-Pad2)
- U9 pad 2: Net-(D2-Pad2) -> GND
- U9 pad 3: Net-(C32-Pad1) -> Net-(R23-Pad2)
Routing:
- net VBAT: track 0.00 -> 171.5 mm, vias 0 -> 2
- net 5V: track 0.00 -> 138.9 mm, vias 0 -> 2
- net GND: track 65.3 -> 202.7 mm, vias 33 -> 77
- net VBAT_ALWON: track 0.00 -> 127.5 mm
- net 2V5: track 0.00 -> 78.1 mm, vias 0 -> 6
- net Net-(BT1-Pad2): track 0.00 -> 67.8 mm
- net 1V1: track 0.00 -> 65.8 mm, vias 0 -> 8
- net VIO: track 5.26 -> 65.5 mm, vias 3 -> 18
- net LCD_BLEN: track 0.00 -> 50.5 mm, vias 0 -> 1
- net Net-(J1-Pad5): track 0.00 -> 20.1 mm
- net Net-(J1-Pad8): track 0.00 -> 19.5 mm, vias 0 -> 1
- net LCD_ID: track 69.2 -> 51.5 mm
- net LCD_DB0: track 66.7 -> 49.2 mm
- net LCD_DB2: track 66.0 -> 48.6 mm
- net LCD_DB4: track 66.6 -> 49.3 mm
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- added copper zone on Pwr.Cu, net 1V1
Other:
- board size 96 x 145.5 mm -> 88 x 137.5 mm
- board text added: "ON ->"
- board text added: "note: coil footprint is random, needs fixing."
- board text removed: "1V1 serdes"
- board text removed: "<- ON"

Commit message: Nearly done...
Parts:
- removed U8: ESP-WROVER32, RF_Module:ESP32-WROOM-32
- added C27: 22p, Capacitor_SMD:C_0603_1608Metric, B.Cu at (127.5, 109.4)
- added J11: Conn_02x06_Odd_Even, Connector_PinSocket_2.54mm:PinSocket_2x06_P2.54mm_Horizontal, F.Cu at (135.5, 36.0)
- added R48: 100, Resistor_SMD:R_0603_1608Metric, B.Cu at (100.7, 97.9)
- added R49: 100, Resistor_SMD:R_0603_1608Metric, B.Cu at (102.0, 101.0)
- added R50: 100, Resistor_SMD:R_0603_1608Metric, B.Cu at (103.2, 97.9)
- added R51: 100, Resistor_SMD:R_0603_1608Metric, B.Cu at (104.5, 101.0)
- added R52: 100, Resistor_SMD:R_0603_1608Metric, B.Cu at (105.8, 98.0)
- added R53: 100, Resistor_SMD:R_0603_1608Metric, B.Cu at (106.8, 101.0)
- added R54: 100, Resistor_SMD:R_0603_1608Metric, B.Cu at (95.2, 135.7)
- C4: footprint Capacitor_SMD:C_0805_2012Metric -> Capacitor_SMD:C_0603_1608Metric
- J2: footprint JeroensFootprints:USB_Micro-B_0.8mm_taobao -> JeroensFootprints:USB_Micro-B_China_MK5P
- J6: value Conn_02x16_Odd_Even -> Conn_02x20_Odd_Even; footprint Connector_PinSocket_2.54mm:PinSocket_2x16_P2.54mm_Horizontal -> Connector_PinSocket_2.54mm:PinSocket_2x20_P2.54mm_Horizontal
- L1: value SWPA252010S4R7MT -> LQH3NPN2R2MJRL; footprint lib:SWPA25xx -> lib:Murata_1212
- L2, L3: footprint Inductor_SMD:L_Murata_DEM35xxC -> lib:Murata_1212
- R21: value 100K -> 82K
- R23: value R -> 560K
- R33, R34, R35, R36, R37, R38: value 100 -> 180
- R47: value R -> 100K
- R6: value R -> 330K
- TP12: moved to B.Cu
- U1: value LFE5UM-45F -> LFE5Ux-45F
- U4: value 25LCxxx -> W25Q128JVSIQ
- moved C11 81.5 mm to (130.9, 106.1), turned to 0 degrees
- moved R23 79.1 mm to (125.9, 109.4), turned to 270 degrees
- moved R22 78.9 mm to (130.8, 102.2)
- moved C26 75.7 mm to (134.5, 106.1)
- moved C10 75.2 mm to (130.9, 104.1), turned to 0 degrees
- moved R47 72.7 mm to (125.9, 112.6), turned to 270 degrees
- moved L2 69.9 mm to (134.3, 113.2), turned to 0 degrees
- moved C31 65.8 mm to (134.5, 119.8), turned to 180 degrees
- moved U9 65.3 mm to (134.3, 109.5), turned to 0 degrees
- moved D1 65.2 mm to (130.2, 111.1), turned to 270 degrees
- moved C4 63.1 mm to (127.8, 122.9), turned to 270 degrees
- moved R21 59.9 mm to (127.8, 126.1), turned to 270 degrees
- moved C33 58.0 mm to (130.6, 117.9), turned to 0 degrees
- moved L3 57.9 mm to (134.5, 126.4), turned to 0 degrees
- moved U7 57.7 mm to (134.5, 122.8), turned to 0 degrees
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Connections:
- net /FPGA/FLASH_HOLD renamed FLASH_HOLD
- net /FPGA/FLASH_MISO renamed FLASH_MISO
- net /FPGA/FLASH_MOSI renamed FLASH_MOSI
- net /FPGA/FLASH_SCK renamed FLASH_SCK
- net /FPGA/FLASH_WP renamed FLASH_WP
- J10 pad 1: (no net) -> SAO2_DRM
- J10 pad 2: (no net) -> SAO2_GPIO3
- J6 pad 10: GENIO_8 -> GENIO_2
- J6 pad 11: GENIO_9 -> GENIO_3
- J6 pad 12: GENIO_10 -> GENIO_4
- J6 pad 13: GENIO_11 -> GENIO_5
- J6 pad 14: GENIO_12 -> GENIO_6
- J6 pad 15: GENIO_13 -> GENIO_7
- J6 pad 16: GENIO_14 -> GENIO_8
- J6 pad 17: GENIO_15 -> GENIO_9
- J6 pad 18: GENIO_16 -> GENIO_10
- J6 pad 19: GENIO_17 -> GENIO_11
- J6 pad 20: GENIO_18 -> GENIO_12
- J6 pad 21: GENIO_19 -> GENIO_13
- J6 pad 22: GENIO_20 -> GENIO_14
- J6 pad 23: GENIO_21 -> GENIO_15
- J6 pad 24: GENIO_22 -> GENIO_16
- J6 pad 25: GENIO_23 -> GENIO_17
- J6 pad 26: GENIO_24 -> GENIO_18
- J6 pad 27: GENIO_25 -> GENIO_19
- J6 pad 28: GENIO_26 -> GENIO_20
- J6 pad 29: GENIO_27 -> GENIO_21
- J6 pad 3: (no net) -> Net-(J6-Pad3)
- J6 pad 30: GENIO_28 -> GENIO_22
- J6 pad 31: GENIO_29 -> GENIO_23
- J6 pad 32: GENIO_30 -> GENIO_24
- J6 pad 4: (no net) -> Net-(J6-Pad4)
- J6 pad 5: (no net) -> Net-(J6-Pad5)
- J6 pad 6: (no net) -> Net-(J6-Pad6)
- J6 pad 7: (no net) -> Net-(J6-Pad7)
- J6 pad 8: (no net) -> Net-(J6-Pad8)
- J6 pad 9: (no net) -> GENIO_1
- J7 pad 1: (no net) -> VIO
- J7 pad 2: (no net) -> GND
- J7 pad 3: (no net) -> SAO1_SCL
- J7 pad 4: (no net) -> SAO1_SDA
- J7 pad 5: (no net) -> SAO1_GPIO2
- J7 pad 6: (no net) -> SAO1_GPIO1
- J8 pad 1: (no net) -> VIO
- J8 pad 2: (no net) -> GND
- J8 pad 3: (no net) -> SAO2_SCL
- J8 pad 4: (no net) -> SAO2_SDA
- J8 pad 5: (no net) -> SAO2_GPIO2
- J8 pad 6: (no net) -> SAO2_GPIO1
- J9 pad 1: (no net) -> SAO1_DRM
- J9 pad 2: (no net) -> SAO1_GPIO3
- R25 pad 1: (no net) -> USB_PU
- U1 pad A10: GENIO_28 -> GENIO_20
- U1 pad A11: GENIO_30 -> GENIO_24
- U1 pad A13: (no net) -> GENIO_28
- U1 pad A14: (no net) -> PMODB_4
- U1 pad A15: (no net) -> PMODA_3
- U1 pad A16: (no net) -> PMODA_1
- U1 pad A17: (no net) -> SAO2_SCL
- U1 pad A18: (no net) -> SAO2_GPIO2
- U1 pad A2: GENIO_12 -> SAO1_GPIO1
- U1 pad A3: GENIO_14 -> SAO1_GPIO2
- U1 pad A4: GENIO_16 -> SAO1_DRM
- U1 pad A5: GENIO_18 -> GENIO_3
- U1 pad A6: GENIO_20 -> GENIO_6
- U1 pad A7: GENIO_22 -> GENIO_9
- U1 pad A8: GENIO_24 -> GENIO_12
- U1 pad A9: GENIO_26 -> GENIO_16
- U1 pad B1: GENIO_9 -> LED6
- U1 pad B10: GENIO_27 -> GENIO_19
- U1 pad B11: GENIO_29 -> GENIO_23
- U1 pad B13: (no net) -> GENIO_27
- U1 pad B15: (no net) -> PMODB_3
- U1 pad B16: (no net) -> PMODB_1
- U1 pad B17: (no net) -> SAO2_GPIO3
- U1 pad B18: (no net) -> SAO2_SDA
- U1 pad B19: (no net) -> SAO2_GPIO1
- U1 pad B2: GENIO_10 -> SAO1_SDA
- U1 pad B3: GENIO_13 -> SAO1_SCL
- U1 pad B4: GENIO_15 -> SAO1_GPIO3
- U1 pad B5: GENIO_17 -> GENIO_2
- U1 pad B6: GENIO_19 -> GENIO_5
- U1 pad B8: GENIO_23 -> GENIO_11
- U1 pad B9: GENIO_25 -> GENIO_15
- U1 pad C10: (no net) -> GENIO_18
- U1 pad C11: (no net) -> GENIO_22
- U1 pad C13: (no net) -> GENIO_26
- U1 pad C14: (no net) -> GENIO_30
- U1 pad C16: (no net) -> PMODA_2
- U1 pad C17: (no net) -> SAO2_DRM
- U1 pad C2: GENIO_8 -> LED5
- U1 pad C3: GENIO_11 -> LED3
- U1 pad C5: LED5 -> GENIO_1
- U1 pad C6: LED6 -> GENIO_4
- U1 pad C7: GENIO_21 -> GENIO_8
- U1 pad C8: (no net) -> GENIO_10
- U1 pad C9: (no net) -> GENIO_14
- U1 pad D10: (no net) -> GENIO_17
- U1 pad D11: (no net) -> GENIO_21
- U1 pad D13: (no net) -> GENIO_25
- U1 pad D14: (no net) -> GENIO_29
- U1 pad D15: (no net) -> PMODA_4
- U1 pad D16: (no net) -> PMODB_2
- U1 pad D3: LED3 -> LED2
- U1 pad D6: (no net) -> GENIO_7
- U1 pad D9: (no net) -> GENIO_13
- U1 pad E3: LED2 -> LED1
- U1 pad E4: (no net) -> USB_PU
- U1 pad F3: LED1 -> USB_D+
- U1 pad F4: (no net) -> USB_VBUSDET
- U1 pad G2: (no net) -> BTN_LEFT
- U1 pad G3: BTN_LEFT -> USB_D-
- U1 pad R1: (no net) -> Net-(R54-Pad1)
- U4 pad 1: /FPGA/FLASH_CS -> (no net)
Routing:
- net SAO2_DRM: track 0.00 -> 125.1 mm, vias 0 -> 2
- net PMODB_4: track 0.00 -> 123.7 mm, vias 0 -> 2
- net PMODB_3: track 0.00 -> 121.9 mm, vias 0 -> 2
- net PMODA_4: track 0.00 -> 121.4 mm, vias 0 -> 2
- net PMODB_2: track 0.00 -> 121.0 mm, vias 0 -> 2
- net SAO2_GPIO3: track 0.00 -> 118.8 mm, vias 0 -> 2
- net SAO2_SCL: track 0.00 -> 116.6 mm, vias 0 -> 2
- net PMODA_3: track 0.00 -> 116.5 mm, vias 0 -> 2
- net SAO2_GPIO2: track 0.00 -> 115.9 mm, vias 0 -> 2
- net SAO2_GPIO1: track 0.00 -> 115.8 mm, vias 0 -> 2
- net PMODA_2: track 0.00 -> 114.6 mm, vias 0 -> 2
- net SAO1_GPIO3: track 0.00 -> 114.4 mm, vias 0 -> 1
- net 5V: track 138.9 -> 251.9 mm, vias 2 -> 3
- net PMODB_1: track 0.00 -> 112.7 mm, vias 0 -> 2
- net SAO1_DRM: track 0.00 -> 112.6 mm, vias 0 -> 3
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Other:
- board text added: "SAO: shroud space?"
- board text removed: "ToDo: replace USB footprint for something sane"
- board text removed: "note: coil footprint is random, needs fixing."
