File: FPGA.sch (KiCad schematic (older format))
At the start: 53 parts, among them J1 Conn_02x04_Odd_Even, U1 LFE5UM-45F, U2 25LCxxx, U8 LY68L6400SLIT, U9 LY68L6400SLIT, X1 X1G004481001400

Commit message: Proto 1
Parts:
- added D10, D5, D6, D7, D8, D9: LED, LED_SMD:LED_0603_1608Metric, symbol Device:LED
- added R41, R42, R43, R44, R45, R46: 470, Resistor_SMD:R_0603_1608Metric, symbol Device:R
- C1: renamed from C52; value C -> 100n
- C2: renamed from C51; value C -> 100n
- R10: renamed from R4; value NS -> 4K7
- R15: renamed from R9; value NS -> 0
- R16: renamed from R10; value 0 -> NS
- R6: renamed from R33; value R -> 0
- R9: renamed from R3; value 4K7 -> NS
- renumbered C46 to C10, C47 to C11, C8 to C12, C10 to C13, C12 to C14, C14 to C15, C22 to C18, C23 to C19, C26 to C20, C57 to C3, C53 to C4, C3 to C6, C4 to C7, C6 to C8, C7 to C9, R37 to R1, R5 to R11, R6 to R12, R7 to R13, R8 to R14, R38 to R2, R39 to R3, R40 to R4, R36 to R5, R1 to R7, R2 to R8, TP6 to TP1, TP15 to TP10, TP1 to TP11, TP7 to TP2, TP8 to TP3, TP9 to TP4, TP10 to TP5, TP11 to TP6, TP12 to TP7, TP13 to TP8, TP14 to TP9, U8 to U2, U9 to U3, U2 to U4
Connections:
- net GND: now also D10.1 (K), D5.1 (K), D6.1 (K), D7.1 (K), D8.1 (K), D9.1 (K)
- net PWMOUT: now also U1.D20 (PR23C/VREF1_2)
- net LED6: now reaches U1.C6 (PT11A)
- net LED6: now also R46.1
- net LED4: now reaches U1.C4 (PL14A)
- net LED4: now also R44.1
- net LED5: now reaches U1.C5 (PL11D)
- net LED5: now also R45.1
- net LED3: now reaches U1.D3 (PL17D)
- net LED3: now also R43.1
- net LED2: now reaches U1.E3 (PL20B)
- net LED2: now also R42.1
- net LED1: now reaches U1.F3 (PL32B/PCLKC7_1)
- net LED1: now also R41.1
- net LCD_BLEN: now reaches U1.H3 (PL29D)
- net VBAT renamed VBAT_ALWON
- new net: D5.2 (A), R41.2
- new net: D6.2 (A), R42.2
- new net: D7.2 (A), R43.2
- new net: D8.2 (A), R44.2
- new net: D9.2 (A), R45.2
- new net: D10.2 (A), R46.2
- no-connect marks 0 -> 111
Other:
- note added: "R6 can be removed to apply different VIO_PSRAM"
- note removed: "R33 can be removed to apply different VIO_PSRAM"

Commit message: New design
Parts:
- U2, U3: footprint Package_SO:SO-8_5.3x6.2mm_P1.27mm -> Package_SO:SSOP-8_3.9x5.05mm_P1.27mm
Connections:
- net BTN_A: now also U1.D1 (PL26B); no longer U1.C9 (PT27A)
- net BTN_B: now also U1.E2 (PL32D/PCLKC7_0); no longer U1.C11 (PT38B/PCLKC0_0)
- net BTN_DOWN: now also U1.C1 (PL26A); no longer U1.T20 (PR62C)
- net BTN_LEFT: now also U1.G3 (PL32A/PCLKT7_1); no longer U1.U19 (PR65C)
- net BTN_RIGHT: now also U1.F2 (PL32C/PCLKT7_0); no longer U1.U20 (PR62D)
- net BTN_SELECT: now also U1.D2 (PL26C); no longer U1.L19 (PR35C/PCLKT3_0)
- net BTN_START: now also U1.E1 (PL26D); no longer U1.C20 (PR23A)
- net BTN_UP: now also U1.F1 (PL35B/PCLKC6_1); no longer U1.U18 (PR68A)
- net CLK: no longer U1.J20 (PR32C/PCLKT2_0)
- net GENIO_1: no longer U1.F1 (PL35B/PCLKC6_1)
- net GENIO_2: no longer U1.F2 (PL32C/PCLKT7_0)
- net GENIO_3: no longer U1.E1 (PL26D)
- net GENIO_4: no longer U1.E2 (PL32D/PCLKC7_0)
- net GENIO_5: no longer U1.D1 (PL26B)
- net GENIO_6: no longer U1.D2 (PL26C)
- net GENIO_7: no longer U1.C1 (PL26A)
- net HDMI_CK+: now also U1.P20 (PR62A); no longer U1.N16 (PR41A)
- net HDMI_CK-: now also U1.R20 (PR62B); no longer U1.M17 (PR41B)
- net HDMI_D1+: now also U1.L20 (PR35A/PCLKT3_1); no longer U1.N17 (PR44A)
- net HDMI_D1-: now also U1.M20 (PR35B/PCLKC3_1); no longer U1.P16 (PR44B/VREF1_3)
- net HDMI_D2+: now also U1.L16 (PR38A/GR_PCLK3_0); no longer U1.P20 (PR62A)
- net HDMI_D2-: now also U1.L17 (PR38B); no longer U1.R20 (PR62B)
- net HDMI_HEAC+: now also U1.T19 (PR65A); no longer U1.L20 (PR35A/PCLKT3_1)
- net HDMI_HEAC-: now also U1.R18 (PR65B); no longer U1.M20 (PR35B/PCLKC3_1)
- net LCD_CS: now also U1.P3 (PL68C/LLC_GPLL0T_IN); no longer U1.J1 (PL41B)
- net LCD_DB0: now also U1.J3 (PL38C/GR_PCLK6_1); no longer U1.P1 (PL68A)
- net LCD_DB1: now also U1.H1 (PL41C); no longer U1.N3 (PL62A)
- net LCD_DB10: now also U1.M4 (PL59A); no longer U1.M3 (PL62B)
- net LCD_DB11: now also U1.L1 (PL65C); no longer U1.K3 (PL38D)
- net LCD_DB12: now also U1.M3 (PL62B); no longer U1.L1 (PL65C)
- net LCD_DB13: now also U1.M1 (PL65B); no longer U1.J3 (PL38C/GR_PCLK6_1)
- net LCD_DB14: now also U1.N4 (PL59C); no longer U1.L2 (PL62D)
- net LCD_DB15: now also U1.N2 (PL65A); no longer U1.H1 (PL41C)
- net LCD_DB16: now also U1.N3 (PL62A); no longer U1.K1 (PL41D)
- net LCD_DB17: now also U1.N1 (PL65D); no longer U1.G2 (PL35A/PCLKT6_1)
- net LCD_DB2: now also U1.K4 (PL44A); no longer U1.P2 (PL68B)
- net LCD_DB3: now also U1.J1 (PL41B); no longer U1.N4 (PL59C)
- net LCD_DB4: now also U1.K3 (PL38D); no longer U1.N1 (PL65D)
- net LCD_DB5: now also U1.K2 (PL41A); no longer U1.M4 (PL59A)
- net LCD_DB6: now also U1.L4 (PL44C); no longer U1.N2 (PL65A)
- net LCD_DB7: now also U1.K1 (PL41D); no longer U1.M5 (PL53A)
- net LCD_DB8: now also U1.L3 (PL62C); no longer U1.M1 (PL65B)
- net LCD_DB9: now also U1.L2 (PL62D); no longer U1.K4 (PL44A)
- net LCD_FMARK: now also U1.G1 (PL35D/PCLKC6_0); no longer U1.P4 (PL68D/LLC_GPLL0C_IN)
- net LCD_ID: now also U1.J4 (PL38A/GR_PCLK6_0); no longer U1.P3 (PL68C/LLC_GPLL0T_IN)
- net LCD_RD: now also U1.P2 (PL68B); no longer U1.H2 (PL35C/PCLKT6_0)
- net LCD_RS: now also U1.P1 (PL68A); no longer U1.G1 (PL35D/PCLKC6_0)
- net LCD_RST: now also U1.H2 (PL35C/PCLKT6_0); no longer U1.P5 (PL59D)
- net LCD_WR: now also U1.P4 (PL68D/LLC_GPLL0C_IN); no longer U1.K2 (PL41A)
- net PWMOUT: no longer U1.D20 (PR23C/VREF1_2)
- net RAM1_CE: now also U1.D20 (PR23C/VREF1_2); no longer U1.A16 (PT74A)
- net RAM1_SCLK: now also U1.E20 (PR26A); no longer U1.A15 (PT67A)
- net RAM1_SIO0: now also U1.E19 (PR23D); no longer U1.B15 (PT69A)
- net RAM1_SIO1: now also U1.D19 (PR23B); no longer U1.B16 (PT74B)
- net RAM1_SIO2: now also U1.C20 (PR23A); no longer U1.A17 (PT80A)
- net RAM1_SIO3: now also U1.F19 (PR26B); no longer U1.A14 (PT56A)
- net RAM2_CE: now also U1.F20 (PR26C); no longer U1.A19 (PT85A/URC_GPLL1T_IN)
- net RAM2_SCLK: now also U1.J19 (PR32A/PCLKT2_1); no longer U1.A18 (PT83A)
- net RAM2_SIO0: now also U1.J20 (PR32C/PCLKT2_0); no longer U1.B18 (PT80B)
- net RAM2_SIO1: now also U1.G19 (PR29A/GR_PCLK2_1); no longer U1.B19 (PT83B)
- net RAM2_SIO2: now also U1.G20 (PR26D); no longer U1.B20 (PT85B/URC_GPLL1C_IN)
- net RAM2_SIO3: now also U1.H20 (PR29B); no longer U1.B17 (PT78A)
- net USB_D+: no longer U1.J19 (PR32A/PCLKT2_1)
- net USB_D-: no longer U1.K19 (PR32B/PCLKC2_1)
- net USB_PU: no longer U1.H20 (PR29B)
- net USB_VBUSDET: no longer U1.G20 (PR26D)
- net VIO: now also U1.F11 (VCCIO1[2]), U1.F12 (VCCIO1[2]); no longer U1.H14 (VCCIO2[3]), U1.H15 (VCCIO2[3]), U1.J15 (VCCIO2[3])
- net VIO_PSRAM: now also U1.H14 (VCCIO2[3]), U1.H15 (VCCIO2[3]), U1.J15 (VCCIO2[3]); no longer U1.F11 (VCCIO1[2]), U1.F12 (VCCIO1[2])
- no-connect marks 111 -> 99
Changed lines of the file:
@@
 EESchema Schematic File Version 4
 LIBS:hadbadge2019-cache
-EELAYER 26 0
+EELAYER 29 0
 EELAYER END
 $Descr A3 16535 11693
@@
 	6900 8550 6900 8850
 Connection ~ 6900 8850
-Text GLabel 1100 6350 0    50   Input ~ 0
+Text GLabel 9450 6450 0    50   Input ~ 0
 VIO
 Text GLabel 3100 6450 0    50   Input ~ 0
@@
 	1    0    0    -1
 $EndComp
+Text GLabel 3100 6050 0    50   Input ~ 0
+LCD_RS
+Text GLabel 3100 6150 0    50   Input ~ 0
+LCD_RD
+Text GLabel 3100 5950 0    50   Input ~ 0
+LCD_DB17
+Text GLabel 3100 5650 0    50   Input ~ 0
+LCD_DB15
+Text GLabel 3100 5850 0    50   Input ~ 0
+LCD_DB13
+Text GLabel 3100 5750 0    50   Input ~ 0
+LCD_DB11
+Text GLabel 3100 5550 0    50   Input ~ 0
+LCD_DB9
+Text GLabel 3100 4250 0    50   Input ~ 0
+LCD_DB7
+Text GLabel 3100 3950 0    50   Input ~ 0
+LCD_DB5
+Text GLabel 3100 4150 0    50   Input ~ 0
+LCD_DB3
+Text GLabel 3100 4050 0    50   Input ~ 0
+LCD_DB1
+Text GLabel 3100 3250 0    50   Input ~ 0
+LCD_RST
 Text GLabel 3100 3450 0    50   Input ~ 0
-LCD_RS
-Text GLabel 3100 3250 0    50   Input ~ 0
-LCD_RD
-Text GLabel 3100 3150 0    50   Input ~ 0
-LCD_DB17
-Text GLabel 3100 4050 0    50   Input ~ 0
-LCD_DB15
+LCD_FMARK
+Text GLabel 3100 6250 0    50   Input ~ 0
+LCD_CS
+Text GLabel 3100 6350 0    50   Input ~ 0
+LCD_WR
+Text GLabel 3100 5250 0    50   Input ~ 0
+LCD_DB16
+Text GLabel 3100 4950 0    50   Input ~ 0
+LCD_DB14
+Text GLabel 3100 5450 0    50   Input ~ 0
+LCD_DB12
+Text GLabel 3100 4850 0    50   Input ~ 0
+LCD_DB10
+Text GLabel 3100 5350 0    50   Input ~ 0
+LCD_DB8
+Text GLabel 3100 4450 0    50   Input ~ 0
+LCD_DB6
+Text GLabel 3100 3850 0    50   Input ~ 0
+LCD_DB4
+Text GLabel 3100 4350 0    50   Input ~ 0
+LCD_DB2
 Text GLabel 3100 3650 0    50   Input ~ 0
-LCD_DB13
-Text GLabel 3100 3850 0    50   Input ~ 0
-LCD_DB11
-Text GLabel 3100 4350 0    50   Input ~ 0
-LCD_DB9
-Text GLabel 3100 4750 0    50   Input ~ 0
-LCD_DB7
-Text GLabel 3100 4850 0    50   Input ~ 0
-LCD_DB5
-Text GLabel 3100 4950 0    50   Input ~ 0
-LCD_DB3
-Text GLabel 3100 5250 0    50   Input ~ 0
-LCD_DB1
-Text GLabel 3100 5150 0    50   Input ~ 0
-LCD_RST
-Text GLabel 3100 6350 0    50   Input ~ 0
-LCD_FMARK
-Text GLabel 3100 4150 0    50   Input ~ 0
-LCD_CS
-Text GLabel 3100 3950 0    50   Input ~ 0
-LCD_WR
-Text GLabel 3100 4250 0    50   Input ~ 0
-LCD_DB16
-Text GLabel 3100 5550 0    50   Input ~ 0
-LCD_DB14
-Text GLabel 3100 5750 0    50   Input ~ 0
-LCD_DB12
-Text GLabel 3100 5450 0    50   Input ~ 0
-LCD_DB10
-Text GLabel 3100 5850 0    50   Input ~ 0
-LCD_DB8
-Text GLabel 3100 5650 0    50   Input ~ 0
-LCD_DB6
-Text GLabel 3100 5950 0    50   Input ~ 0
-LCD_DB4
-Text GLabel 3100 6150 0    50   Input ~ 0
-LCD_DB2
-Text GLabel 3100 6050 0    50   Input ~ 0
 LCD_DB0
-Text GLabel 3100 6250 0    50   Input ~ 0
+Text GLabel 3100 3550 0    50   Input ~ 0
 LCD_ID
-Text GLabel 7150 3450 0    50   Input ~ 0
+Text GLabel 3100 3350 0    50   Input ~ 0
 BTN_UP
-Text GLabel 7150 4150 0    50   Input ~ 0
+Text GLabel 5050 5150 0    50   Input ~ 0
 BTN_DOWN
-Text GLabel 7150 3750 0    50   Input ~ 0
+Text GLabel 5050 5950 0    50   Input ~ 0
 BTN_LEFT
-Text GLabel 7150 3950 0    50   Input ~ 0
+Text GLabel 5050 6050 0    50   Input ~ 0
 BTN_RIGHT
-Text GLabel 3100 3350 0    50   Input ~ 0
+Text GLabel 2400 2850 0    50   Input ~ 0
 GENIO_1
-Text GLabel 5050 5450 0    50   Input ~ 0
+Text GLabel 5450 6700 0    50   Input ~ 0
 GENIO_3
-Text GLabel 5050 5350 0    50   Input ~ 0
+Text GLabel 4600 7150 0    50   Input ~ 0
 GENIO_5
-Text GLabel 5050 5150 0    50   Input ~ 0
+Text GLabel 5100 7000 0    50   Input ~ 0
 GENIO_7
 Text GLabel 5050 4950 0    50   Input ~ 0
@@
 Text GLabel 5050 5050 0    50   Input ~ 0
 GENIO_8
-Text GLabel 5050 5250 0    50   Input ~ 0
+Text GLabel 4600 7050 0    50   Input ~ 0
 GENIO_6
-Text GLabel 5050 6250 0    50   Input ~ 0
+Text GLabel 5700 6600 0    50   Input ~ 0
 GENIO_4
-Text GLabel 5050 6050 0    50   Input ~ 0
+Text GLabel 4950 6700 0    50   Input ~ 0
 GENIO_2
-Text GLabel 7150 4250 0    50   Input ~ 0
-HDMI_D2+
-Text GLabel 7150 4050 0    50   Input ~ 0
-HDMI_D2-
-Text GLabel 7150 5150 0    50   Input ~ 0
-HDMI_D1+
-Text GLabel 7150 4950 0    50   Input ~ 0
-HDMI_D1-
 Text GLabel 7150 4650 0    50   Input ~ 0
 HDMI_D0+
 Text GLabel 7150 4450 0    50   Input ~ 0
 HDMI_D0-
-Text GLabel 7150 5550 0    50   Input ~ 0
+Text GLabel 7150 4250 0    50   Input ~ 0
 HDMI_CK+
-Text GLabel 7150 5350 0    50   Input ~ 0
+Text GLabel 7150 4050 0    50   Input ~ 0
 HDMI_CK-
-Text GLabel 7150 6350 0    50   Input ~ 0
+Text GLabel 7150 3850 0    50   Input ~ 0
 HDMI_HEAC+
-Text GLabel 7150 6150 0    50   Input ~ 0
+Text GLabel 7150 3650 0    50   Input ~ 0
 HDMI_HEAC-
-Text GLabel 1100 3350 0    50   Input ~ 0
+Text GLabel 1050 2950 0    50   Input ~ 0
 CLK
-Text GLabel 1100 3450 0    50   Input ~ 0
+Text GLabel 900  2550 0    50   Input ~ 0
 USB_D+
-Text GLabel 1100 3250 0    50   Input ~ 0
+Text GLabel 900  2450 0    50   Input ~ 0
 USB_D-
-Text GLabel 1100 3650 0    50   Input ~ 0
+Text GLabel 1100 2700 0    50   Input ~ 0
 USB_PU
-Text GLabel 1100 3950 0    50   Input ~ 0
+Text GLabel 1050 2350 0    50   Input ~ 0
 USB_VBUSDET
 $Comp
@@
 F 0 "U2" H 9800 2100 50  0000 C CNN
 F 1 "LY68L6400SLIT" H 9550 2200 50  0000 C CNN
-F 2 "Package_SO:SO-8_5.3x6.2mm_P1.27mm" H 9950 1700 50  0001 C CNN
+F 2 "Package_SO:SSOP-8_3.9x5.05mm_P1.27mm" H 9950 1700 50  0001 C CNN
 F 3 "https://datasheet.lcsc.com/szlcsc/Lyontek-Inc-LY68L6400SLIT_C261881.pdf" H 9950 1700 50  0001 C CNN
 	1    10000 1750
@@
 F 0 "U3" H 12100 2100 50  0000 C CNN
 F 1 "LY68L6400SLIT" H 11950 2200 50  0000 C CNN
-F 2 "Package_SO:SO-8_5.3x6.2mm_P1.27mm" H 12300 1700 50  0001 C CNN
+F 2 "Package_SO:SSOP-8_3.9x5.05mm_P1.27mm" H 12300 1700 50  0001 C CNN
 F 3 "https://datasheet.lcsc.com/szlcsc/Lyontek-Inc-LY68L6400SLIT_C261881.pdf" H 12300 1700 50  0001 C CNN
 	1    12350 1750
@@
 Text GLabel 9300 6900 2    50   Input ~ 0
 VIO_PSRAM
-Text GLabel 9450 6450 0    50   Input ~ 0
+Text GLabel 1100 6350 0    50   Input ~ 0
 VIO_PSRAM
 Text GLabel 10000 1250 1    50   Input ~ 0
@@
 Text GLabel 11800 1800 0    50   Input ~ 0
 RAM2_SCLK
-Text GLabel 9450 3550 0    50   Input ~ 0
+Text GLabel 1100 3350 0    50   Input ~ 0
 RAM2_SIO0
-Text GLabel 9450 3250 0    50   Input ~ 0
+Text GLabel 1100 3850 0    50   Input ~ 0
 RAM2_SIO1
-Text GLabel 9450 3150 0    50   Input ~ 0
-RAM2_SIO2
-Text GLabel 9450 3850 0    50   Input ~ 0
-RAM2_SIO3
 Text GLabel 13700 1250 1    50   Input ~ 0
 VIO_PSRAM
@@
 Text Notes 9100 6750 0    50   ~ 0
 R6 can be removed to apply different VIO_PSRAM
-Text GLabel 9450 3350 0    50   Input ~ 0
+Text GLabel 1100 4150 0    50   Input ~ 0
 RAM2_CE
-Text GLabel 9450 3450 0    50   Input ~ 0
+Text GLabel 1100 3450 0    50   Input ~ 0
 RAM2_SCLK
-Text GLabel 9450 4250 0    50   Input ~ 0
+Text GLabel 1100 4550 0    50   Input ~ 0
 RAM1_CE
-Text GLabel 9450 4750 0    50   Input ~ 0
+Text GLabel 1100 4250 0    50   Input ~ 0
 RAM1_SCLK
-Text GLabel 9450 4650 0    50   Input ~ 0
+Text GLabel 1100 4350 0    50   Input ~ 0
 RAM1_SIO0
-Text GLabel 9450 4050 0    50   Input ~ 0
-RAM1_SIO1
-Text GLabel 9450 3750 0    50   Input ~ 0
+Text GLabel 1100 4650 0    50   Input ~ 0
 RAM1_SIO2
-Text GLabel 9450 5150 0    50   Input ~ 0
+Text GLabel 1100 4050 0    50   Input ~ 0
 RAM1_SIO3
 Text GLabel 12950 1600 2    50   Input ~ 0
@@
 Text GLabel 12950 1900 2    50   Input ~ 0
 RAM2_SIO3
-Text GLabel 11650 4150 0    50   Input ~ 0
+Text GLabel 5050 5350 0    50   Input ~ 0
 BTN_A
-Text GLabel 11650 3150 0    50   Input ~ 0
+Text GLabel 5050 6250 0    50   Input ~ 0
 BTN_B
-Text GLabel 7150 6250 0    50   Input ~ 0
+Text GLabel 5050 5250 0    50   Input ~ 0
 BTN_SELECT
-Text GLabel 1100 4650 0    50   Input ~ 0
+Text GLabel 5050 5450 0    50   Input ~ 0
 BTN_START
 Wire Wire Line
@@
 NoConn ~ 1100 3550
 NoConn ~ 1100 3750
-NoConn ~ 1100 3850
-NoConn ~ 1100 4050
-NoConn ~ 1100 4150
-NoConn ~ 1100 4250
-NoConn ~ 1100 4350
-NoConn ~ 1100 4450
 NoConn ~ 1100 4750
 NoConn ~ 1100 4850
@@
 NoConn ~ 1100 6150
 NoConn ~ 1100 6250
-NoConn ~ 3100 5350
 NoConn ~ 3100 5050
 NoConn ~ 3100 4650
 NoConn ~ 3100 4550
-NoConn ~ 3100 4450
 NoConn ~ 3100 3750
-NoConn ~ 3100 3550
 NoConn ~ 5050 3950
 NoConn ~ 5050 4150
@@
 NoConn ~ 5050 5650
 NoConn ~ 5050 5750
-NoConn ~ 5050 5950
 NoConn ~ 7150 6050
 NoConn ~ 7150 5950
@@
 NoConn ~ 7150 4550
 NoConn ~ 7150 4350
-NoConn ~ 7150 3850
-NoConn ~ 7150 3650
 NoConn ~ 7150 3550
 NoConn ~ 7150 3350
@@
 	1    0    0    -1
 $EndComp
-Text GLabel 1100 4550 0    50   Input ~ 0
+Text GLabel 1100 2850 0    50   Input ~ 0
 PWMOUT
 Text GLabel 5050 5850 0    50   Input ~ 0
 LCD_BLEN
+Text GLabel 7150 5950 0    50   Input ~ 0
+HDMI_D2+
+Text GLabel 7150 5750 0    50   Input ~ 0
+HDMI_D2-
+Text GLabel 7150 6150 0    50   Input ~ 0
+HDMI_D1-
+Text GLabel 7150 6350 0    50   Input ~ 0
+HDMI_D1+
+Text GLabel 1100 3950 0    50   Input ~ 0
+RAM2_SIO2
+Text GLabel 1100 3650 0    50   Input ~ 0
+RAM2_SIO3
+Text GLabel 1100 4450 0    50   Input ~ 0
+RAM1_SIO1
 $EndSCHEMATC

Commit message: WiP for proto 2
Parts:
- removed C10, C11, C4: 100n, Capacitor_SMD:C_0603_1608Metric, symbol Device:C
- removed R6: 0, Resistor_SMD:R_0603_1608Metric, symbol Device:R
- removed TP1, TP10, TP2, TP3, TP4, TP5, TP6, TP7, TP8, TP9: TestPoint, TestPoint:TestPoint_Pad_D1.0mm, symbol Connector:TestPoint
- added U8: ESP-WROVER32, RF_Module:ESP32-WROOM-32, symbol jeroens_components:ESP-WROVER32
Connections:
- net labels removed: 1V1_SERDES, VIO_PSRAM
- wire segments 112 -> 109
- no-connect marks 99 -> 109
Other:
- note removed: "R6 can be removed to apply different VIO_PSRAM"

Commit message: Nearly done...
Parts:
- removed U8: ESP-WROVER32, RF_Module:ESP32-WROOM-32, symbol jeroens_components:ESP-WROVER32
- added R54: 100, Resistor_SMD:R_0603_1608Metric, symbol Device:R
- U1: value LFE5UM-45F -> LFE5Ux-45F
- U1: value LFE5UM-45F -> LFE5Ux-45F; Notes (none) -> Lattice LFE5U-45F-8BG381C or LFE5UM-45F-8BG381C
- U2, U3: Notes (none) -> Lyontek
- U4: value 25LCxxx -> W25Q128JVSIQ
- X1: Notes (none) -> Seiko-Epson
Connections:
- net labels added: FLASH_CS_INT, PMODA_1, PMODA_2, PMODA_3, PMODA_4, PMODB_1, PMODB_2, PMODB_3, PMODB_4, SAO1_DRM, SAO1_GPIO1, SAO1_GPIO2, SAO1_GPIO3, SAO1_SCL, SAO1_SDA, SAO2_DRM, SAO2_GPIO1, SAO2_GPIO2, SAO2_GPIO3, SAO2_SCL, SAO2_SDA
- wire segments 109 -> 106
- no-connect marks 109 -> 91
Other:
- note added: "ToDo: mux to mux CS between internal and external"

Commit message: Proto2, final version
Parts:
- removed J1: Conn_02x04_Odd_Even, Connector_PinHeader_2.54mm:PinHeader_2x04_P2.54mm_Vertical, symbol Connector_Generic:Conn_02x04_Odd_Even
- added C28: 100n, Capacitor_SMD:C_0603_1608Metric, symbol Device:C_Small
- added C29: 100n, Capacitor_SMD:C_0603_1608Metric, symbol Device:C
- added C30: 10n, Capacitor_SMD:C_0603_1608Metric, symbol Device:C_Small
- added D11, D12, D13, D14, D15: LED, LED_SMD:LED_0603_1608Metric, symbol Device:LED
- added J1: Conn_02x05_Odd_Even, Connector_PinHeader_2.54mm:PinHeader_2x05_P2.54mm_Vertical, symbol Connector_Generic:Conn_02x05_Odd_Even
- added R55, R56: 4K7, Resistor_SMD:R_0603_1608Metric, symbol Device:R
- added R57: 100, Resistor_SMD:R_0603_1608Metric, symbol Device:R
- added R60: NS, Resistor_SMD:R_0603_1608Metric, symbol Device:R
- added R61, R62, R63, R64, R65: 470, Resistor_SMD:R_0603_1608Metric, symbol Device:R
- added TP1, TP2, TP3, TP4, TP5, TP6: TestPoint, TestPoint:TestPoint_Pad_D1.0mm, symbol Connector:TestPoint
- added U11: 74LVC1G175, Package_TO_SOT_SMD:SOT-23-6, symbol 74xGxx:74LVC1G175
- added U8: 74LVC1G3157, Package_TO_SOT_SMD:SOT-23-6, symbol 74xGxx:74LVC1G3157
- D10, D5, D8: Notes (none) -> RED
- D6, D7, D9: Notes (none) -> YELLOW
Connections:
- net CLK: now also U1.U18 (PR68A), TP2.1
- net FLASH_CS: now also U8.4; no longer R7.1
- net FLASH_CS_INT: now also R7.2, U8.1
- net GENIO_25: now also U1.G18 (PR17B); no longer U1.D13 (PT53A)
- net GENIO_26: now also U1.H17 (PR20B); no longer U1.C13 (PT51B)
- net GENIO_27: now also U1.B12 (PT44A/PCLKT1_0); no longer U1.B13 (PT51A)
- net GENIO_28: now also U1.A12 (PT49A); no longer U1.A13 (PT49B)
- net GENIO_29: now also U1.E17 (PR14B); no longer U1.D14 (PT58A)
- net GND: now also C28.2, C29.2, C30.2, D11.1 (K), D12.1 (K), D13.1 (K), D14.1 (K), D15.1 (K), J1.2 (Pin_2), U11.2 (GND), U8.2 (GND)
- net PMODA_1: now also U1.A15 (PT67A); no longer U1.A16 (PT74A)
- net PMODA_3: now also U1.A14 (PT56A); no longer U1.A15 (PT67A)
- net PMODA_4: now also U1.D16 (PT76B); no longer U1.D15 (PT71A)
- net PMODB_1: now also U1.B15 (PT69A); no longer U1.B16 (PT74B)
- net PMODB_2: now also U1.C15 (PT69B); no longer U1.D16 (PT76B)
- net PMODB_3: now also U1.A13 (PT49B); no longer U1.B15 (PT69A)
- net PMODB_4: now also U1.B13 (PT51A); no longer U1.A14 (PT56A)
- net PWMOUT: now also U1.T1 (PB4B/D6/IO6)
- net SAO2_GPIO1: now also U1.B18 (PT80B); no longer U1.B19 (PT83B)
- net SAO2_GPIO2: now also U1.A17 (PT80A); no longer U1.A18 (PT83A)
- net SAO2_GPIO3: now also U1.B16 (PT74B); no longer U1.B17 (PT78A)
- net SAO2_SCL: now also U1.A16 (PT74A); no longer U1.A17 (PT80A)
- net SAO2_SDA: now also U1.B17 (PT78A); no longer U1.B18 (PT80B)
- net VBAT_ALWON: now also J1.1 (Pin_1)
- net ADCREFOUT: now reaches U1.A19 (PT85A/URC_GPLL1T_IN)
- net ADCREFOUT: now also R57.2
- net LED7: now reaches U1.B20 (PT85B/URC_GPLL1C_IN)
- net LED7: now also R63.1
- net at U1.C12 (PT44B/PCLKC1_0): now also TP6.1
- net ADCREF: now reaches U1.C18 (PR11A/URC_GPLL0T_IN)
- net ADCREF: now also U1.D18 (PR14A), U1.F17 (PR17A), U1.H18 (PR20A), C30.1, R57.1
- net ADC4: now reaches U1.D17 (PR11B/URC_GPLL0C_IN)
- net at U1.T18 (PR65D): now also TP5.1
- net at U1.U17 (PR68B): now also TP1.1
- net at U1.U19 (PR65C): now also TP3.1
- net at U1.U20 (PR62D): now also TP4.1
- net FSEL_D: now reaches U1.D5 (PL17B)
- net FSEL_D: now also U11.3 (D)
- net FSEL_C: now reaches U1.E5 (PL20C)
- net FSEL_C: now also U11.1 (C)
- net DBGTX: now reaches U1.U1 (PB6A/D5/MISO2/IO5)
- net DBGTX: now also J1.9 (Pin_9)
- net DBGRX: now reaches U1.U2 (PB13B/CS1N)
- net DBGRX: now also J1.10 (Pin_10)
- net at R2.2, U1.R5 (TDI): now also J1.5 (Pin_5)
- net at R4.1, U1.T5 (TCK): now also J1.8 (Pin_8)
- net at R1.2, U1.U5 (TMS): now also J1.7 (Pin_7)
- net at R3.2, U1.V4 (TDO): now also J1.6 (Pin_6)
- net VIO renamed VCC
- net VCC: now also R7.1, C29.1, J1.3 (Pin_3), R55.1, R56.2, R60.1, R62.1, U11.5 (VCC), U8.5 (VCC); no longer R7.2
- new net: U11.4 (Q), U8.6
- new net: C28.1, R55.2, U11.6 (~CLR)
- new net: D11.2 (A), R61.2
- new net: R60.2, R61.1
- new net: D12.2 (A), R62.2
- new net: D13.2 (A), R63.2
- new net: D14.2 (A), R64.2
- new net: D15.2 (A), R65.2
- new net FLASH_CS_EXT: R56.1, U8.3
- new net LED8: R64.1, U1.B19 (PT83B)
- new net LED9: R65.1, U1.A18 (PT83A)
- no-connect marks 91 -> 79
Other:
- note added: "ToDo: check footprints"
- note removed: "ToDo: mux to mux CS between internal and external"
- moved on the sheet: R4
