File: FPGA.sch (KiCad schematic (older format))
At the start: 77 parts, among them J1 Conn_02x05_Odd_Even, U1 LFE5Ux-45F, U11 74LVC1G175, U2 LY68L6400SLIT, U3 LY68L6400SLIT, U4 W25Q128JVSIQ, U8 74LVC1G3157, X1 X1G004481001400

Commit message: Fix fab drawings to make sense
Parts:
- D10, D11, D5, D8: value LED -> LED RED; Notes RED -> (none)
- D12, D13, D6, D9: value LED -> LED YELLOW; Notes YELLOW -> (none)
- D14, D15: value LED -> LED GREEN; Notes GREEN -> (none)
- D7: value LED -> LED YELLOW
Connections:
- no-connect marks 79 -> 82
Changed lines of the file:
@@
 NoConn ~ 5050 5750
 NoConn ~ 7150 6050
-NoConn ~ 7150 5950
 NoConn ~ 7150 5850
-NoConn ~ 7150 5750
 NoConn ~ 7150 5650
 NoConn ~ 7150 5450
@@
 NoConn ~ 7150 3250
 NoConn ~ 7150 3150
-NoConn ~ 9450 4150
 NoConn ~ 9450 4350
-NoConn ~ 9450 4450
 NoConn ~ 9450 4850
 NoConn ~ 9450 5250
 NoConn ~ 9450 5750
-NoConn ~ 9450 5850
 NoConn ~ 9450 5950
-NoConn ~ 9450 6050
 NoConn ~ 9450 6150
-NoConn ~ 9450 6250
 NoConn ~ 11650 5650
 NoConn ~ 11650 5350
@@
 NoConn ~ 11650 4250
 NoConn ~ 11650 3950
-NoConn ~ 7500 8150
-NoConn ~ 7500 8250
 NoConn ~ 7500 8350
 NoConn ~ 7500 8850
-NoConn ~ 7500 9050
 NoConn ~ 7500 9150
 NoConn ~ 7500 9250
@@
 P 14100 5800
 F 0 "D5" V 14138 5683 50  0000 R CNN
-F 1 "LED" V 14047 5683 50  0000 R CNN
+F 1 "LED RED" H 13950 5950 50  0000 R CNN
 F 2 "LED_SMD:LED_0603_1608Metric" H 14100 5800 50  0001 C CNN
 F 3 "~" H 14100 5800 50  0001 C CNN
-F 4 "RED" H 14100 5800 50  0001 C CNN "Notes"
 	1    14100 5800
 	0    -1   -1   0
@@
 P 14450 5800
 F 0 "D6" V 14488 5683 50  0000 R CNN
-F 1 "LED" V 14397 5683 50  0000 R CNN
+F 1 "LED YELLOW" H 14450 5900 50  0000 R CNN
 F 2 "LED_SMD:LED_0603_1608Metric" H 14450 5800 50  0001 C CNN
 F 3 "~" H 14450 5800 50  0001 C CNN
-F 4 "YELLOW" H 14450 5800 50  0001 C CNN "Notes"
 	1    14450 5800
 	0    -1   -1   0
@@
 P 14800 5800
 F 0 "D7" V 14838 5683 50  0000 R CNN
-F 1 "LED" V 14747 5683 50  0000 R CNN
+F 1 "LED YELLOW" H 14800 5900 50  0000 R CNN
 F 2 "LED_SMD:LED_0603_1608Metric" H 14800 5800 50  0001 C CNN
 F 3 "~" H 14800 5800 50  0001 C CNN
@@
 P 15150 5800
 F 0 "D8" V 15188 5683 50  0000 R CNN
-F 1 "LED" V 15097 5683 50  0000 R CNN
+F 1 "LED RED" H 15000 5900 50  0000 R CNN
 F 2 "LED_SMD:LED_0603_1608Metric" H 15150 5800 50  0001 C CNN
 F 3 "~" H 15150 5800 50  0001 C CNN
-F 4 "RED" H 15150 5800 50  0001 C CNN "Notes"
 	1    15150 5800
 	0    -1   -1   0
@@
 P 15450 5800
 F 0 "D9" V 15488 5683 50  0000 R CNN
-F 1 "LED" V 15397 5683 50  0000 R CNN
+F 1 "LED YELLOW" H 15450 5900 50  0000 R CNN
 F 2 "LED_SMD:LED_0603_1608Metric" H 15450 5800 50  0001 C CNN
 F 3 "~" H 15450 5800 50  0001 C CNN
-F 4 "YELLOW" H 15450 5800 50  0001 C CNN "Notes"
 	1    15450 5800
 	0    -1   -1   0
@@
 P 15750 5800
 F 0 "D10" V 15788 5683 50  0000 R CNN
-F 1 "LED" V 15697 5683 50  0000 R CNN
+F 1 "LED RED" H 15600 5900 50  0000 R CNN
 F 2 "LED_SMD:LED_0603_1608Metric" H 15750 5800 50  0001 C CNN
 F 3 "~" H 15750 5800 50  0001 C CNN
-F 4 "RED" H 15750 5800 50  0001 C CNN "Notes"
 	1    15750 5800
 	0    -1   -1   0
@@
 P 14050 7600
 F 0 "D11" V 14088 7483 50  0000 R CNN
-F 1 "LED" V 13997 7483 50  0000 R CNN
+F 1 "LED RED" H 13950 7700 50  0000 R CNN
 F 2 "LED_SMD:LED_0603_1608Metric" H 14050 7600 50  0001 C CNN
 F 3 "~" H 14050 7600 50  0001 C CNN
-F 4 "RED" H 14050 7600 50  0001 C CNN "Notes"
 	1    14050 7600
 	0    -1   -1   0
@@
 P 14400 7600
 F 0 "D12" V 14438 7483 50  0000 R CNN
-F 1 "LED" V 14347 7483 50  0000 R CNN
+F 1 "LED YELLOW" H 14400 7700 50  0000 R CNN
 F 2 "LED_SMD:LED_0603_1608Metric" H 14400 7600 50  0001 C CNN
 F 3 "~" H 14400 7600 50  0001 C CNN
-F 4 "YELLOW" H 14400 7600 50  0001 C CNN "Notes"
 	1    14400 7600
 	0    -1   -1   0
@@
 P 14750 7600
 F 0 "D13" V 14788 7483 50  0000 R CNN
-F 1 "LED" V 14697 7483 50  0000 R CNN
+F 1 "LED YELLOW" H 14750 7700 50  0000 R CNN
 F 2 "LED_SMD:LED_0603_1608Metric" H 14750 7600 50  0001 C CNN
 F 3 "~" H 14750 7600 50  0001 C CNN
-F 4 "YELLOW" H 14750 7600 50  0001 C CNN "Notes"
 	1    14750 7600
 	0    -1   -1   0
@@
 P 15100 7600
 F 0 "D14" V 15138 7483 50  0000 R CNN
-F 1 "LED" V 15047 7483 50  0000 R CNN
+F 1 "LED GREEN" H 15050 7700 50  0000 R CNN
 F 2 "LED_SMD:LED_0603_1608Metric" H 15100 7600 50  0001 C CNN
 F 3 "~" H 15100 7600 50  0001 C CNN
-F 4 "GREEN" H 15100 7600 50  0001 C CNN "Notes"
 	1    15100 7600
 	0    -1   -1   0
@@
 P 15400 7600
 F 0 "D15" V 15438 7483 50  0000 R CNN
-F 1 "LED" V 15347 7483 50  0000 R CNN
+F 1 "LED GREEN" H 15350 7700 50  0000 R CNN
 F 2 "LED_SMD:LED_0603_1608Metric" H 15400 7600 50  0001 C CNN
 F 3 "~" H 15400 7600 50  0001 C CNN
-F 4 "GREEN" H 15400 7600 50  0001 C CNN "Notes"
 	1    15400 7600
 	0    -1   -1   0
@@
 	0    -1   -1   0
 $EndComp
+NoConn ~ 1100 3250
+NoConn ~ 5050 5850
+NoConn ~ 7150 4950
+NoConn ~ 7150 5150
+NoConn ~ 7150 5350
+NoConn ~ 7150 5550
+NoConn ~ 7150 6250
+NoConn ~ 9450 5450
+NoConn ~ 9450 5350
+NoConn ~ 9450 5050
+NoConn ~ 9450 4550
+NoConn ~ 3100 4750
+NoConn ~ 7150 4150
 $EndSCHEMATC

Commit message: This is proto 3.
Parts:
- removed D10, D11, D5, D8: LED RED, LED_SMD:LED_0603_1608Metric, symbol Device:LED
- removed D12, D13, D6, D7, D9: LED YELLOW, LED_SMD:LED_0603_1608Metric, symbol Device:LED
- removed D14, D15: LED GREEN, LED_SMD:LED_0603_1608Metric, symbol Device:LED
- added D10, D11, D12, D13, D14, D15, D5, D6, D7, D8, D9: FC-B1010RGBT-HG, lib:FC-B1010RGBT-HG, symbol FC-B1010RGBT-HG:FC-B1010RGBT-HG
- added Q3, Q4, Q5: AO3400, Package_TO_SOT_SMD:SOT-23, symbol jeroens_components:AO3400
- added R66, R67: 4K7, Resistor_SMD:R_0603_1608Metric, symbol Device:R
- added R69, R70, R71: 10K, Resistor_SMD:R_0603_1608Metric, symbol Device:R
- added TP7: TestPoint, TestPoint:TestPoint_Pad_D1.0mm, symbol Connector:TestPoint
- R41, R42, R43, R44, R45, R46, R61, R62, R63, R64, R65: value 470 -> 220R
- X1: footprint Crystal:Crystal_SMD_7050-4Pin_7.0x5.0mm -> lib:Seiko_fp_crystal_SMD_7050-4Pin_7.0x5.0mm
Connections:
- net FLASH_CS_EXT: now also U8.1; no longer U8.3
- net FLASH_CS_INT: now also U8.3; no longer U8.1
- net FSEL_C: now also R67.1
- net FSEL_D: now also R66.1
- net GND: now also Q3.2 (S), Q4.2 (S), Q5.2 (S), R66.2, R67.2, R69.2, R70.2, R71.2
- net VCC: no longer R60.1, R62.1
- net at U1.J16 (PR20D): now also TP7.1
- net LEDB: now reaches U1.K18 (PR29D)
- net LEDB: now also Q5.1 (G), R71.1
- net LED11: now reaches U1.K19 (PR32B/PCLKC2_1)
- net LED11: now also R62.1
- net LED10: now reaches U1.K20 (PR32D/PCLKC2_0)
- net LED10: now also R60.1
- net LEDG: now reaches U1.L18 (PR38C/GR_PCLK3_1)
- net LEDG: now also Q4.1 (G), R70.1
- net LEDR: now reaches U1.P19 (PR59C)
- net LEDR: now also Q3.1 (G), R69.1
- net IRDA_TX: now reaches U1.R16 (PR44C)
- net IRDA_SD: now reaches U1.T16 (PR53A)
- net IRDA_RX: now reaches U1.U16 (PR68C/LRC_GPLL0T_IN)
- net at R41.2: now also D5.1 (A)
- net at R42.2: now also D6.1 (A)
- net at R43.2: now also D7.1 (A)
- net at R44.2: now also D8.1 (A)
- net at R45.2: now also D9.1 (A)
- net at R46.2: now also D10.1 (A)
- net at R61.2: now also D11.1 (A)
- net at R62.2: now also D12.1 (A)
- net at R63.2: now also D13.1 (A)
- net at R64.2: now also D14.1 (A)
- net at R65.2: now also D15.1 (A)
- new net CATB: D10.4 (BK), D11.4 (BK), D12.4 (BK), D13.4 (BK), D14.4 (BK), D15.4 (BK), D5.4 (BK), D6.4 (BK), D7.4 (BK), D8.4 (BK), D9.4 (BK), Q5.3 (D)
- new net CATG: D10.3 (GK), D11.3 (GK), D12.3 (GK), D13.3 (GK), D14.3 (GK), D15.3 (GK), D5.3 (GK), D6.3 (GK), D7.3 (GK), D8.3 (GK), D9.3 (GK), Q4.3 (D)
- new net CATR: D10.2 (RK), D11.2 (RK), D12.2 (RK), D13.2 (RK), D14.2 (RK), D15.2 (RK), D5.2 (RK), D6.2 (RK), D7.2 (RK), D8.2 (RK), D9.2 (RK), Q3.3 (D)
- no-connect marks 82 -> 73
Other:
- note added: "Bridge pads of\nR60 for extra\nhack-o-meter\ncreds"
- note added: "Note: All LEDs indeed are RGB LEDs, but the default\nconfig only shows some fixed colors. Good luck\ngetting full control!\n"
- note added: "Rec: min 32MBit for '45F FPGA\n(bitstream is 10MBit with max blockram)"
- note removed: "Rec: 32MBit for '45F FPGA\n(bitstream is 10MBit with max blockram)"
- note removed: "ToDo: check footprints"
- moved on the sheet: C29, R41, R56, R60, R7, U1I

Commit message: Starting to add fixes for final ver
Parts:
- added R72: 1K, Resistor_SMD:R_0603_1608Metric, symbol Device:R
- R57: value 100 -> 1K
Connections:
- net CATB: now also D10.3 (GK), D11.3 (GK), D12.2 (RK), D13.2 (RK), D14.3 (GK), D15.3 (GK), D5.3 (GK), D6.3 (GK), D7.3 (GK), D8.3 (GK), D9.3 (GK), Q4.3 (D); no longer D10.4 (BK), D11.4 (BK), D12.4 (BK), D13.4 (BK), D14.4 (BK), D15.4 (BK), D5.4 (BK), D6.4 (BK), D7.4 (BK), D8.4 (BK), D9.4 (BK), Q5.3 (D)
- net GENIO_25: now also U1.F18 (PR14D)
- net GENIO_26: now also U1.H16 (PR17D)
- net GENIO_29: now also U1.E16 (PR11C)
- net GND: no longer R69.2
- net LED11: now also R72.2
- net LEDR: now also R69.2; no longer R69.1
- net VCC: now also R69.1, R72.1
- removed net CATG: D10.3 (GK), D11.3 (GK), D12.3 (GK), D13.3 (GK), D14.3 (GK), D15.3 (GK), D5.3 (GK), D6.3 (GK), D7.3 (GK), D8.3 (GK), D9.3 (GK), Q4.3 (D)
- net CATR renamed CATA
- net CATA: now also D10.4 (BK), D11.4 (BK), D12.3 (GK), D13.3 (GK), D6.4 (BK), D8.4 (BK); no longer D10.2 (RK), D11.2 (RK), D12.2 (RK), D13.2 (RK), D6.2 (RK), D8.2 (RK)
- new net CATC: D10.2 (RK), D11.2 (RK), D12.4 (BK), D13.4 (BK), D14.4 (BK), D15.4 (BK), D5.4 (BK), D6.2 (RK), D7.4 (BK), D8.2 (RK), D9.4 (BK), Q5.3 (D)
- no-connect marks 73 -> 70
Other:
- note added: "Bridge pads of\nR60 (or use 0R \nresistor) for extra\nhack-o-meter\ncreds"
- note added: "Note: All LEDs indeed are RGB LEDs, but normally, \nonly CATA is powered so all LEDs will only light up \nin whatever color is connected to that. Good luck \ngetting full RGB!"
- note removed: "Bridge pads of\nR60 for extra\nhack-o-meter\ncreds"
- note removed: "Note: All LEDs indeed are RGB LEDs, but the default\nconfig only shows some fixed colors. Good luck\ngetting full control!\n"
- moved on the sheet: R69
Changed lines of the file:
@@
-$Comp
-L ECP5UM45:LFE5UM-45F U1
-U 3 1 5C5E9B3D
-P 1100 3150
-F 0 "U1" H 2450 1750 60  0000 L CNN
-F 1 "LFE5Ux-45F" H 2450 1650 60  0000 L CNN
-F 2 "lib:Lattice_caBGA-381_17.0x17.0mm_Layout20x20_P0.8mm_Ball0.4mm_Pad0.4mm_NSMD" H 1100 3150 50  0001 C CNN
-F 3 "" H 1100 3150 50  0001 C CNN
-	3    1100 3150
-	1    0    0    -1
-$EndComp
 $Comp
 L ECP5UM45:LFE5UM-45F U1
@@
 NoConn ~ 1100 3750
 NoConn ~ 1100 4950
-NoConn ~ 1100 5150
 NoConn ~ 1100 5350
-NoConn ~ 1100 5550
 NoConn ~ 1100 5750
 NoConn ~ 1100 5950
-NoConn ~ 1100 6050
 NoConn ~ 3100 5050
 NoConn ~ 3100 4650
@@
 P 7950 7000
 F 0 "R57" V 7743 7000 50  0000 C CNN
-F 1 "100" V 7834 7000 50  0000 C CNN
+F 1 "1K" V 7834 7000 50  0000 C CNN
 F 2 "Resistor_SMD:R_0603_1608Metric" V 7880 7000 50  0001 C CNN
 F 3 "~" H 7950 7000 50  0001 C CNN
@@
 IRDA_SD
 Text GLabel 13650 3550 3    50   Input ~ 0
-CATR
+CATA
 Text GLabel 13850 3550 3    50   Input ~ 0
-CATG
+CATB
 Text GLabel 14050 3550 3    50   Input ~ 0
-CATB
+CATC
 Text GLabel 13850 2850 1    50   Input ~ 0
 LED1
@@
 	1    0    0    -1
 $EndComp
+Text GLabel 14850 3550 3    50   Input ~ 0
+CATA
+Text GLabel 14650 3550 3    50   Input ~ 0
+CATB
 Text GLabel 14450 3550 3    50   Input ~ 0
-CATR
-Text GLabel 14650 3550 3    50   Input ~ 0
-CATG
-Text GLabel 14850 3550 3    50   Input ~ 0
-CATB
+CATC
 Text GLabel 14650 2850 1    50   Input ~ 0
 LED2
@@
 $EndComp
 Text GLabel 15250 3550 3    50   Input ~ 0
-CATR
+CATA
 Text GLabel 15450 3550 3    50   Input ~ 0
-CATG
+CATB
 Text GLabel 15650 3550 3    50   Input ~ 0
-CATB
+CATC
 Text GLabel 15450 2850 1    50   Input ~ 0
 LED3
@@
 	1    0    0    -1
 $EndComp
+Text GLabel 14050 4900 3    50   Input ~ 0
+CATA
+Text GLabel 13850 4900 3    50   Input ~ 0
+CATB
 Text GLabel 13650 4900 3    50   Input ~ 0
-CATR
-Text GLabel 13850 4900 3    50   Input ~ 0
-CATG
-Text GLabel 14050 4900 3    50   Input ~ 0
-CATB
+CATC
 Text GLabel 13850 4200 1    50   Input ~ 0
 LED4
@@
 $EndComp
 Text GLabel 14450 4900 3    50   Input ~ 0
-CATR
+CATA
 Text GLabel 14650 4900 3    50   Input ~ 0
-CATG
+CATB
 Text GLabel 14850 4900 3    50   Input ~ 0
-CATB
+CATC
 Text GLabel 14650 4200 1    50   Input ~ 0
 LED5
@@
 	1    0    0    -1
 $EndComp
+Text GLabel 15650 4900 3    50   Input ~ 0
+CATA
+Text GLabel 15450 4900 3    50   Input ~ 0
+CATB
 Text GLabel 15250 4900 3    50   Input ~ 0
-CATR
-Text GLabel 15450 4900 3    50   Input ~ 0
-CATG
-Text GLabel 15650 4900 3    50   Input ~ 0
-CATB
+CATC
 Text GLabel 15450 4200 1    50   Input ~ 0
 LED6
@@
 	1    0    0    -1
 $EndComp
+Text GLabel 14050 6650 3    50   Input ~ 0
+CATA
+Text GLabel 13850 6650 3    50   Input ~ 0
+CATB
 Text GLabel 13650 6650 3    50   Input ~ 0
-CATR
-Text GLabel 13850 6650 3    50   Input ~ 0
-CATG
-Text GLabel 14050 6650 3    50   Input ~ 0
-CATB
+CATC
 Text GLabel 13850 5550 1    50   Input ~ 0
 LED10
@@
 	1    0    0    -1
 $EndComp
+Text GLabel 14650 6650 3    50   Input ~ 0
+CATA
 Text GLabel 14450 6650 3    50   Input ~ 0
-CATR
-Text GLabel 14650 6650 3    50   Input ~ 0
-CATG
+CATB
 Text GLabel 14850 6650 3    50   Input ~ 0
-CATB
-Text GLabel 14650 5950 1    50   Input ~ 0
+CATC
+Text GLabel 14650 5550 1    50   Input ~ 0
 LED11
 $Comp
@@
 	1    0    0    -1
 $EndComp
+Text GLabel 15450 6650 3    50   Input ~ 0
+CATA
 Text GLabel 15250 6650 3    50   Input ~ 0
-CATR
-Text GLabel 15450 6650 3    50   Input ~ 0
-CATG
+CATB
 Text GLabel 15650 6650 3    50   Input ~ 0
-CATB
+CATC
 Text GLabel 15450 5950 1    50   Input ~ 0
 LED7
@@
 $EndComp
 Text GLabel 13650 8000 3    50   Input ~ 0
-CATR
+CATA
 Text GLabel 13850 8000 3    50   Input ~ 0
-CATG
+CATB
 Text GLabel 14050 8000 3    50   Input ~ 0
-CATB
+CATC
 Text GLabel 13850 7300 1    50   Input ~ 0
 LED8
@@
 $EndComp
 Text GLabel 14450 8000 3    50   Input ~ 0
-CATR
+CATA
 Text GLabel 14650 8000 3    50   Input ~ 0
-CATG
+CATB
 Text GLabel 14850 8000 3    50   Input ~ 0
-CATB
+CATC
 Text GLabel 14650 7300 1    50   Input ~ 0
 LED9
@@
 	13850 5850 13850 5950
 Text Notes 13500 2400 0    50   ~ 0
-Note: All LEDs indeed are RGB LEDs, but the default\nconfig only shows some fixed colors. Good luck\ngetting full control!\n
+Note: All LEDs indeed are RGB LEDs, but normally, \nonly CATA is powered so all LEDs will only light up \nin whatever color is connected to that. Good luck \ngetting full RGB!
 $Comp
 L jeroens_components:AO3400 Q3
@@
 L Device:R R69
 U 1 1 5D8F8182
-P 13100 9400
-F 0 "R69" H 12850 9400 50  0000 L CNN
-F 1 "10K" H 12850 9300 50  0000 L CNN
-F 2 "Resistor_SMD:R_0603_1608Metric" V 13030 9400 50  0001 C CNN
-F 3 "~" H 13100 9400 50  0001 C CNN
-	1    13100 9400
-	1    0    0    -1
-$EndComp
-$Comp
-L power:GND #PWR0119
-U 1 1 5D8F87E2
-P 13100 9550
-F 0 "#PWR0119" H 13100 9300 50  0001 C CNN
-F 1 "GND" H 13105 9377 50  0000 C CNN
-F 2 "" H 13100 9550 50  0001 C CNN
-F 3 "" H 13100 9550 50  0001 C CNN
-	1    13100 9550
+P 13100 9100
+F 0 "R69" H 12850 9200 50  0000 L CNN
+F 1 "10K" H 12850 9100 50  0000 L CNN
+F 2 "Resistor_SMD:R_0603_1608Metric" V 13030 9100 50  0001 C CNN
+F 3 "~" H 13100 9100 50  0001 C CNN
+	1    13100 9100
 	1    0    0    -1
 $EndComp
@@
 Connection ~ 13100 9250
 Text GLabel 13400 9050 1    50   Input ~ 0
-CATR
+CATA
 $Comp
 L jeroens_components:AO3400 Q4
@@
 Connection ~ 14250 9250
 Text GLabel 14550 9050 1    50   Input ~ 0
-CATG
+CATB
 $Comp
 L jeroens_components:AO3400 Q5
@@
 Connection ~ 15350 9250
 Text GLabel 15650 9050 1    50   Input ~ 0
-CATB
+CATC
 Text GLabel 1100 3550 0    50   Input ~ 0
 LEDB
@@
 	0    -1   -1   0
 $EndComp
-Text Notes 13100 5850 0    50   ~ 0
-Bridge pads of\nR60 for extra\nhack-o-meter\ncreds
+Text Notes 13050 5950 0    50   ~ 0
+Bridge pads of\nR60 (or use 0R \nresistor) for extra\nhack-o-meter\ncreds
+Text GLabel 13100 8950 1    50   Input ~ 0
+VIO
+Text GLabel 14450 5550 1    50   Input ~ 0
+VIO
+$Comp
+L Device:R R72
+U 1 1 5D9EBC23
+P 14450 5700
+F 0 "R72" H 14250 5750 50  0000 L CNN
+F 1 "1K" H 14250 5650 50  0000 L CNN
+F 2 "Resistor_SMD:R_0603_1608Metric" V 14380 5700 50  0001 C CNN
+F 3 "~" H 14450 5700 50  0001 C CNN
+	1    14450 5700
+	1    0    0    -1
+$EndComp
+Wire Wire Line
+	14450 5850 14450 5950
+Wire Wire Line
+	14450 5950 14650 5950
+Wire Wire Line
+	14650 5950 14650 5550
+Connection ~ 14650 5950
+Text GLabel 1100 5150 0    50   Input ~ 0
+GENIO_26
+$Comp
+L ECP5UM45:LFE5UM-45F U1
+U 3 1 5C5E9B3D
+P 1100 3150
+F 0 "U1" H 2450 1750 60  0000 L CNN
+F 1 "LFE5Ux-45F" H 2450 1650 60  0000 L CNN
+F 2 "lib:Lattice_caBGA-381_17.0x17.0mm_Layout20x20_P0.8mm_Ball0.4mm_Pad0.4mm_NSMD" H 1100 3150 50  0001 C CNN
+F 3 "" H 1100 3150 50  0001 C CNN
+	3    1100 3150
+	1    0    0    -1
+$EndComp
+Text GLabel 1100 5550 0    50   Input ~ 0
+GENIO_25
+Text GLabel 1100 6050 0    50   Input ~ 0
+GENIO_29
 $EndSCHEMATC
